File: nRF52832_reference/kicad/nRF52832_qfaa_nfc/nRF52832_qfaa_nfc.sch (KiCad schematic (older format))
At the start: 20 parts, among them X1 32MHz, X2 32.768kHz

Commit message: Save work in progress. Working on NFC connector footprint
Parts:
- added J1: NFC, nRF52:FPC_05P-05mm-RA-SMD_Alt, symbol CONN_01X05
- X2: footprint Crystals:Crystal_SMD_2012-2pin_2.0x1.2mm -> Crystals:Crystal_SMD_3215-2pin_3.2x1.5mm
- nRF1: renamed from nRF?; footprint nRF52840:UQFN-48-1EP_6x6mm_Pitch0.4mm -> nRF52:UQFN-48-1EP_6x6mm_Pitch0.4mm
Connections:
- net GND: now also nRF1.49 (GND)
- net NFC1: now also J1.2 (P2)
- net NFC2: now also J1.4 (P4)
- net P0.00/XL1: now reaches C11.1, X2.1, nRF1.2 (P0.00/XL1)
- net P0.01/XL2: now reaches C12.1, X2.2, nRF1.3 (P0.01/XL2)
- no-connect marks 0 -> 3
Changed lines of the file:
@@
 EELAYER 25 0
 EELAYER END
-$Descr A4 11693 8268
+$Descr USLetter 11000 8500
 encoding utf-8
 Sheet 1 1
 Title ""
-Date ""
-Rev ""
+Date "2017-07-22"
+Rev "0.9"
 Comp ""
 Comment1 ""
@@
 VDD_nRF
 $Comp
-L PWR_FLAG #FLG?
+L PWR_FLAG #FLG01
 U 1 1 59739DE8
 P 2150 1700
-F 0 "#FLG?" H 2150 1775 50  0001 C CNN
+F 0 "#FLG01" H 2150 1775 50  0001 C CNN
 F 1 "PWR_FLAG" H 2150 1850 50  0000 C CNN
 F 2 "" H 2150 1700 50  0001 C CNN
@@
 $EndComp
 $Comp
-L GND #PWR?
+L GND #PWR02
 U 1 1 59739DEA
-P 4200 2050
-F 0 "#PWR?" H 4200 1800 50  0001 C CNN
-F 1 "GND" H 4200 1900 50  0000 C CNN
-F 2 "" H 4200 2050 50  0001 C CNN
-F 3 "" H 4200 2050 50  0001 C CNN
-	1    4200 2050
+P 4200 2100
+F 0 "#PWR02" H 4200 1850 50  0001 C CNN
+F 1 "GND" H 4200 1950 50  0000 C CNN
+F 2 "" H 4200 2100 50  0001 C CNN
+F 3 "" H 4200 2100 50  0001 C CNN
+	1    4200 2100
 	1    0    0    -1
 $EndComp
@@
 $EndComp
 $Comp
-L GND #PWR?
+L GND #PWR03
 U 1 1 59739DED
-P 3650 2050
-F 0 "#PWR?" H 3650 1800 50  0001 C CNN
-F 1 "GND" H 3650 1900 50  0000 C CNN
-F 2 "" H 3650 2050 50  0001 C CNN
-F 3 "" H 3650 2050 50  0001 C CNN
-	1    3650 2050
+P 3650 2100
+F 0 "#PWR03" H 3650 1850 50  0001 C CNN
+F 1 "GND" H 3650 1950 50  0000 C CNN
+F 2 "" H 3650 2100 50  0001 C CNN
+F 3 "" H 3650 2100 50  0001 C CNN
+	1    3650 2100
 	1    0    0    -1
 $EndComp
@@
 $EndComp
 $Comp
-L GND #PWR?
+L GND #PWR04
 U 1 1 59739DF0
 P 4150 5350
-F 0 "#PWR?" H 4150 5100 50  0001 C CNN
+F 0 "#PWR04" H 4150 5100 50  0001 C CNN
 F 1 "GND" H 4150 5200 50  0000 C CNN
 F 2 "" H 4150 5350 50  0001 C CNN
@@
 $EndComp
 $Comp
-L GND #PWR?
+L GND #PWR05
 U 1 1 59739DF7
 P 6200 2000
-F 0 "#PWR?" H 6200 1750 50  0001 C CNN
+F 0 "#PWR05" H 6200 1750 50  0001 C CNN
 F 1 "GND" H 6200 1850 50  0000 C CNN
 F 2 "" H 6200 2000 50  0001 C CNN
@@
 F 0 "X2" V 2500 2950 50  0000 C CNN
 F 1 "32.768kHz" V 2650 3050 50  0000 C CNN
-F 2 "Crystals:Crystal_SMD_2012-2pin_2.0x1.2mm" H 2550 2800 50  0001 C CNN
+F 2 "Crystals:Crystal_SMD_3215-2pin_3.2x1.5mm" H 2550 2800 50  0001 C CNN
 F 3 "" H 2550 2800 50  0001 C CNN
 	1    2550 2800
@@
 $EndComp
 $Comp
-L GND #PWR?
+L GND #PWR06
 U 1 1 59739DFB
 P 1850 3150
-F 0 "#PWR?" H 1850 2900 50  0001 C CNN
+F 0 "#PWR06" H 1850 2900 50  0001 C CNN
 F 1 "GND" H 1850 3000 50  0000 C CNN
 F 2 "" H 1850 3150 50  0001 C CNN
@@
 $EndComp
 $Comp
-L GND #PWR?
+L GND #PWR07
 U 1 1 59739DFE
 P 9450 3150
-F 0 "#PWR?" H 9450 2900 50  0001 C CNN
+F 0 "#PWR07" H 9450 2900 50  0001 C CNN
 F 1 "GND" H 9450 3000 50  0000 C CNN
 F 2 "" H 9450 3150 50  0001 C CNN
@@
 $EndComp
 $Comp
-L GND #PWR?
+L GND #PWR08
 U 1 1 59739E01
 P 6950 2000
-F 0 "#PWR?" H 6950 1750 50  0001 C CNN
+F 0 "#PWR08" H 6950 1750 50  0001 C CNN
 F 1 "GND" H 6950 1850 50  0000 C CNN
 F 2 "" H 6950 2000 50  0001 C CNN
@@
 $EndComp
 $Comp
-L GND #PWR?
+L GND #PWR09
 U 1 1 59739E03
 P 7500 3950
-F 0 "#PWR?" H 7500 3700 50  0001 C CNN
+F 0 "#PWR09" H 7500 3700 50  0001 C CNN
 F 1 "GND" H 7500 3800 50  0000 C CNN
 F 2 "" H 7500 3950 50  0001 C CNN
@@
 $EndComp
 $Comp
-L GND #PWR?
+L GND #PWR010
 U 1 1 59739E0C
 P 5350 1150
-F 0 "#PWR?" H 5350 900 50  0001 C CNN
+F 0 "#PWR010" H 5350 900 50  0001 C CNN
 F 1 "GND" H 5350 1000 50  0000 C CNN
 F 2 "" H 5350 1150 50  0001 C CNN
@@
 	3800 3150 4150 3150
 Wire Wire Line
-	2650 3950 2900 3950
-Wire Wire Line
-	2900 3950 4150 3950
-Wire Wire Line
-	2650 3850 2900 3850
-Wire Wire Line
-	2900 3850 4150 3850
+	2650 3950 4150 3950
+Wire Wire Line
+	2650 3850 4150 3850
 Wire Wire Line
 	3800 3750 4150 3750
@@
 	5750 2050 5750 2150
 Wire Wire Line
-	1600 1800 1800 1800
-Wire Wire Line
-	1800 1800 2150 1800
+	1600 1800 2150 1800
 Wire Wire Line
 	2150 1800 2150 1700
@@
 Connection ~ 1800 1800
 Wire Wire Line
-	4200 2050 4200 2000
-Wire Wire Line
-	4200 1450 4200 1600
-Wire Wire Line
-	4200 1600 4200 1700
+	4200 2000 4200 2100
+Wire Wire Line
+	4200 1450 4200 1700
 Wire Wire Line
 	4850 2000 4850 2150
 Connection ~ 4200 1600
 Wire Wire Line
-	3650 2050 3650 2000
+	3650 2100 3650 2000
 Wire Wire Line
 	3650 1700 3650 1600
@@
 	4000 2850 4150 2850
 Wire Wire Line
-	4150 4750 4150 4850
-Wire Wire Line
-	4150 4850 4150 4950
+	4150 4750 4150 4950
 Wire Wire Line
 	4850 4650 4850 4850
@@
 	4150 5350 4150 5250
 Wire Wire Line
-	6200 1400 6200 1500
-Wire Wire Line
-	6200 1500 6200 1600
+	6200 1400 6200 1600
 Connection ~ 6200 1500
 Wire Wire Line
 	6200 1900 6200 2000
 Wire Wire Line
-	2250 2600 2550 2600
-Wire Wire Line
-	2550 2600 3050 2600
+	2250 2600 3050 2600
 Wire Wire Line
 	2550 2600 2550 2700
@@
 	2550 2900 2550 3050
 Wire Wire Line
-	2250 3050 2550 3050
-Wire Wire Line
-	2550 3050 3400 3050
+	2250 3050 4150 3050
 Wire Wire Line
 	4150 2950 3050 2950
@@
 Connection ~ 2550 2600
 Wire Wire Line
-	4150 3050 3400 3050
-Wire Wire Line
 	3400 3050 3400 3050
 Connection ~ 2550 3050
 Wire Wire Line
-	1850 2600 1850 3050
-Wire Wire Line
-	1850 3050 1850 3150
+	1850 2600 1850 3150
 Wire Wire Line
 	1850 2600 1950 2600
@@
 Connection ~ 1850 3050
 Wire Wire Line
-	6650 3050 8650 3050
-Wire Wire Line
-	8650 3050 8950 3050
+	6650 3050 8950 3050
 Wire Wire Line
 	8650 3050 8650 2850
@@
 	8650 2550 8650 2400
 Wire Wire Line
-	8100 2400 8650 2400
-Wire Wire Line
-	8650 2400 8950 2400
+	8100 2400 8950 2400
 Wire Wire Line
 	9250 2400 9450 2400
 Wire Wire Line
-	9450 2400 9450 3050
-Wire Wire Line
-	9450 3050 9450 3150
+	9450 2400 9450 3150
 Wire Wire Line
 	9250 3050 9450 3050
@@
 Connection ~ 8650 3050
 Wire Wire Line
-	7500 3850 7500 3900
-Wire Wire Line
-	7500 3900 7500 3950
-Wire Wire Line
-	6650 3450 7500 3450
-Wire Wire Line
-	7500 3450 7700 3450
+	7500 3850 7500 3950
+Wire Wire Line
+	6650 3450 7700 3450
 Wire Wire Line
 	7500 3450 7500 3550
@@
 	4950 1700 4950 2150
 Wire Wire Line
-	4750 750  5050 750
-Wire Wire Line
-	5050 750  5350 750
+	4750 750  5350 750
 Wire Wire Line
 	4750 750  4750 900
 Wire Wire Line
-	5350 1050 5350 1100
-Wire Wire Line
-	5350 1100 5350 1150
+	5350 1050 5350 1150
 Wire Wire Line
 	5150 2150 5150 1100
@@
 $EndComp
 $Comp
-L GND #PWR?
+L GND #PWR011
 U 1 1 59739E0E
 P 8900 2700
-F 0 "#PWR?" H 8900 2450 50  0001 C CNN
+F 0 "#PWR011" H 8900 2450 50  0001 C CNN
 F 1 "GND" H 8900 2550 50  0000 C CNN
 F 2 "" H 8900 2700 50  0001 C CNN
@@
 	8900 2700 8850 2700
 $Comp
-L GND #PWR?
+L GND #PWR012
 U 1 1 59739E0F
 P 8400 2700
-F 0 "#PWR?" H 8400 2450 50  0001 C CNN
+F 0 "#PWR012" H 8400 2450 50  0001 C CNN
 F 1 "GND" H 8400 2550 50  0000 C CNN
 F 2 "" H 8400 2700 50  0001 C CNN
@@
 NFC1
 $Comp
-L GND #PWR?
+L GND #PWR013
 U 1 1 59739E14
 P 2900 4450
-F 0 "#PWR?" H 2900 4200 50  0001 C CNN
+F 0 "#PWR013" H 2900 4200 50  0001 C CNN
 F 1 "GND" H 2900 4300 50  0000 C CNN
 F 2 "" H 2900 4450 50  0001 C CNN
@@
 	2900 4450 2900 4350
 $Comp
-L GND #PWR?
+L GND #PWR014
 U 1 1 59739E15
 P 2900 3350
-F 0 "#PWR?" H 2900 3100 50  0001 C CNN
+F 0 "#PWR014" H 2900 3100 50  0001 C CNN
 F 1 "GND" H 2900 3200 50  0000 C CNN
 F 2 "" H 2900 3350 50  0001 C CNN
@@
 	8300 3450 8300 3450
 $Comp
-L nRF52832 nRF?
+L nRF52832 nRF1
 U 1 1 59739DE6
 P 5400 3400
-F 0 "nRF?" H 5400 3600 60  0000 C CNN
+F 0 "nRF1" H 5400 3600 60  0000 C CNN
 F 1 "nRF52832" H 5400 3400 60  0000 C CNN
-F 2 "nRF52840:UQFN-48-1EP_6x6mm_Pitch0.4mm" H 5400 3400 60  0001 C CNN
+F 2 "nRF52:UQFN-48-1EP_6x6mm_Pitch0.4mm" H 5400 3400 60  0001 C CNN
 F 3 "" H 5400 3400 60  0001 C CNN
 	1    5400 3400
@@
 	7250 3150 6650 3150
 $Comp
-L GND #PWR?
+L GND #PWR015
 U 1 1 5973CAAA
 P 7450 2000
-F 0 "#PWR?" H 7450 1750 50  0001 C CNN
+F 0 "#PWR015" H 7450 1750 50  0001 C CNN
 F 1 "GND" H 7450 1850 50  0000 C CNN
 F 2 "" H 7450 2000 50  0001 C CNN
@@
 DEC1
 $Comp
-L +3.3V #PWR?
+L +3.3V #PWR016
 U 1 1 5973FB66
 P 4200 1450
-F 0 "#PWR?" H 4200 1300 50  0001 C CNN
+F 0 "#PWR016" H 4200 1300 50  0001 C CNN
 F 1 "+3.3V" H 4200 1590 50  0000 C CNN
 F 2 "" H 4200 1450 50  0001 C CNN
@@
 $EndComp
 $Comp
-L +3.3V #PWR?
+L +3.3V #PWR017
 U 1 1 5973FC37
 P 1800 1700
-F 0 "#PWR?" H 1800 1550 50  0001 C CNN
+F 0 "#PWR017" H 1800 1550 50  0001 C CNN
 F 1 "+3.3V" H 1800 1840 50  0000 C CNN
 F 2 "" H 1800 1700 50  0001 C CNN
@@
 $EndComp
 $Comp
-L +3.3V #PWR?
+L +3.3V #PWR018
 U 1 1 5973FE1C
 P 4150 4750
-F 0 "#PWR?" H 4150 4600 50  0001 C CNN
+F 0 "#PWR018" H 4150 4600 50  0001 C CNN
 F 1 "+3.3V" H 4150 4890 50  0000 C CNN
 F 2 "" H 4150 4750 50  0001 C CNN
@@
 $EndComp
 $Comp
-L +3.3V #PWR?
+L +3.3V #PWR019
 U 1 1 5973FF85
 P 6200 1400
-F 0 "#PWR?" H 6200 1250 50  0001 C CNN
+F 0 "#PWR019" H 6200 1250 50  0001 C CNN
 F 1 "+3.3V" H 6200 1540 50  0000 C CNN
 F 2 "" H 6200 1400 50  0001 C CNN
@@
 	1    0    0    -1
 $EndComp
+Text Label 2550 2600 0    60   ~ 0
+P0.00/XL1
+Text Label 2550 3050 0    60   ~ 0
+P0.01/XL2
+Wire Wire Line
+	4750 2150 4750 2050
+Wire Wire Line
+	4750 2050 4200 2050
+Connection ~ 4200 2050
+$Comp
+L CONN_01X05 J1
+U 1 1 59742685
+P 2350 3900
+F 0 "J1" H 2350 4200 50  0000 C CNN
+F 1 "NFC" V 2450 3900 50  0000 C CNN
+F 2 "nRF52:FPC_05P-05mm-RA-SMD_Alt" H 2350 3900 50  0001 C CNN
+F 3 "" H 2350 3900 50  0001 C CNN
+	1    2350 3900
+	-1   0    0    -1
+$EndComp
+Wire Wire Line
+	2550 3800 2650 3800
+Wire Wire Line
+	2650 3800 2650 3850
+Wire Wire Line
+	2650 3950 2650 4000
+Wire Wire Line
+	2650 4000 2550 4000
+NoConn ~ 2550 3700
+NoConn ~ 2550 3900
+NoConn ~ 2550 4100
 $EndSCHEMATC
