File: nRF52832_reference/kicad/nRF52832_qfaa_nfc/nRF52832_qfaa_nfc.sch (KiCad schematic (older format))
At the start: 21 parts, among them J1 NFC, X1 32MHz, X2 32.768kHz

Commit message: Reference Project nRF52832_qfaa_nfc ready
Parts:
- removed J1: NFC, nRF52:FPC_05P-05mm-RA-SMD_Alt, symbol CONN_01X05
- added MK1, MK2, MK3, MK4: Mounting_Hole, Nordic_misc:MountingHole_3mm, symbol Mounting_Hole
- added NFC1: NFC_ANTENNA, Nordic_misc:Nordic_misc-NFC_ANT, symbol NFC_ANTENNA
Connections:
- net NFC1: now also NFC1.2 (NFC1)
- net NFC2: now also NFC1.1 (NFC2)
- no-connect marks 3 -> 1
Changed lines of the file:
@@
 EESchema Schematic File Version 2
 LIBS:nRF52832_qfaa_nfc-rescue
-LIBS:nrf52
 LIBS:74xgxx
 LIBS:74xx
@@
 LIBS:zetex
 LIBS:Zilog
+LIBS:Nordic_misc
+LIBS:Nordic_nRF
 LIBS:nRF52832_qfaa_nfc-cache
 EELAYER 25 0
@@
 	3800 3150 4150 3150
 Wire Wire Line
-	2650 3950 4150 3950
-Wire Wire Line
-	2650 3850 4150 3850
+	2550 3950 4150 3950
+Wire Wire Line
+	2550 3850 4150 3850
 Wire Wire Line
 	3800 3750 4150 3750
@@
 	4750 2050 4200 2050
 Connection ~ 4200 2050
-$Comp
-L CONN_01X05 J1
-U 1 1 59742685
-P 2350 3900
-F 0 "J1" H 2350 4200 50  0000 C CNN
-F 1 "NFC" V 2450 3900 50  0000 C CNN
-F 2 "nRF52:FPC_05P-05mm-RA-SMD_Alt" H 2350 3900 50  0001 C CNN
-F 3 "" H 2350 3900 50  0001 C CNN
-	1    2350 3900
-	-1   0    0    -1
-$EndComp
-Wire Wire Line
-	2550 3800 2650 3800
-Wire Wire Line
-	2650 3800 2650 3850
-Wire Wire Line
-	2650 3950 2650 4000
-Wire Wire Line
-	2650 4000 2550 4000
 NoConn ~ 2550 3700
-NoConn ~ 2550 3900
-NoConn ~ 2550 4100
+$Comp
+L Mounting_Hole MK1
+U 1 1 597CF176
+P 8950 1200
+F 0 "MK1" H 8950 1400 50  0000 C CNN
+F 1 "Mounting_Hole" H 8950 1325 50  0000 C CNN
+F 2 "Nordic_misc:MountingHole_3mm" H 8950 1200 50  0001 C CNN
+F 3 "" H 8950 1200 50  0001 C CNN
+	1    8950 1200
+	1    0    0    -1
+$EndComp
+$Comp
+L Mounting_Hole MK3
+U 1 1 597CF2FD
+P 9500 1200
+F 0 "MK3" H 9500 1400 50  0000 C CNN
+F 1 "Mounting_Hole" H 9500 1325 50  0000 C CNN
+F 2 "Nordic_misc:MountingHole_3mm" H 9500 1200 50  0001 C CNN
+F 3 "" H 9500 1200 50  0001 C CNN
+	1    9500 1200
+	1    0    0    -1
+$EndComp
+$Comp
+L Mounting_Hole MK2
+U 1 1 597CF36C
+P 8950 1550
+F 0 "MK2" H 8950 1750 50  0000 C CNN
+F 1 "Mounting_Hole" H 8950 1675 50  0000 C CNN
+F 2 "Nordic_misc:MountingHole_3mm" H 8950 1550 50  0001 C CNN
+F 3 "" H 8950 1550 50  0001 C CNN
+	1    8950 1550
+	1    0    0    -1
+$EndComp
+$Comp
+L Mounting_Hole MK4
+U 1 1 597CF3E8
+P 9500 1550
+F 0 "MK4" H 9500 1750 50  0000 C CNN
+F 1 "Mounting_Hole" H 9500 1675 50  0000 C CNN
+F 2 "Nordic_misc:MountingHole_3mm" H 9500 1550 50  0001 C CNN
+F 3 "" H 9500 1550 50  0001 C CNN
+	1    9500 1550
+	1    0    0    -1
+$EndComp
+$Comp
+L NFC_ANTENNA NFC1
+U 1 1 597D020B
+P 2050 3750
+F 0 "NFC1" H 2050 3700 39  0000 C CNN
+F 1 "NFC_ANTENNA" H 2150 4120 45  0000 R TNN
+F 2 "Nordic_misc:Nordic_misc-NFC_ANT" H 2080 3900 20  0001 C CNN
+F 3 "" H 2050 3750 60  0001 C CNN
+	1    2050 3750
+	-1   0    0    1
+$EndComp
 $EndSCHEMATC

Commit message: Update nRF52832_reference
Parts:
- X1: footprint Crystals:Crystal_SMD_2016-4pin_2.0x1.6mm -> Nordic_nRF:Crystal_SMD_2016-4pin_2.0x1.6mm
- X2: footprint Crystals:Crystal_SMD_3215-2pin_3.2x1.5mm -> Nordic_nRF:Crystal_SMD_3215-2pin_3.2x1.5mm
- nRF1: footprint nRF52:UQFN-48-1EP_6x6mm_Pitch0.4mm -> Nordic_nRF:Nordic_nRF-QFN40P600X600X90-48_N
Changed lines of the file:
@@
 LIBS:Nordic_nRF
 LIBS:nRF52832_qfaa_nfc-cache
-EELAYER 25 0
+EELAYER 26 0
 EELAYER END
 $Descr USLetter 11000 8500
@@
 F 0 "X2" V 2500 2950 50  0000 C CNN
 F 1 "32.768kHz" V 2650 3050 50  0000 C CNN
-F 2 "Crystals:Crystal_SMD_3215-2pin_3.2x1.5mm" H 2550 2800 50  0001 C CNN
+F 2 "Nordic_nRF:Crystal_SMD_3215-2pin_3.2x1.5mm" H 2550 2800 50  0001 C CNN
 F 3 "" H 2550 2800 50  0001 C CNN
 	1    2550 2800
@@
 F 0 "X1" V 8450 2500 50  0000 L CNN
 F 1 "32MHz" V 8550 2300 50  0000 L CNN
-F 2 "Crystals:Crystal_SMD_2016-4pin_2.0x1.6mm" H 8650 2700 50  0001 C CNN
+F 2 "Nordic_nRF:Crystal_SMD_2016-4pin_2.0x1.6mm" H 8650 2700 50  0001 C CNN
 F 3 "" H 8650 2700 50  0001 C CNN
 	1    8650 2700
@@
 F 0 "nRF1" H 5400 3600 60  0000 C CNN
 F 1 "nRF52832" H 5400 3400 60  0000 C CNN
-F 2 "nRF52:UQFN-48-1EP_6x6mm_Pitch0.4mm" H 5400 3400 60  0001 C CNN
+F 2 "Nordic_nRF:Nordic_nRF-QFN40P600X600X90-48_N" H 5400 3400 60  0001 C CNN
 F 3 "" H 5400 3400 60  0001 C CNN
 	1    5400 3400
