File: nRF52832_reference/kicad/nRF52832_qfaa_nfc/nRF52832_qfaa_nfc.kicad_pcb (KiCad board)
At the start: 2 copper layers, 40 x 34 mm, 21 parts, among them J1 NFC, X1 32MHz, X2 32.768kHz

Commit message: Save work in progress before working on RF Antenna
Parts:
- moved J1 4.00 mm to (94.2, 117.1)
Routing:
- net /NFC1: track 14.0 -> 18.0 mm
- net /NFC2: track 12.8 -> 16.8 mm
Other:
- board size 40 x 34 mm -> 40 x 40 mm
Changed lines of the file:
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@@
     (links 60)
     (no_connects 0)
-    (area 78.674999 81.674999 118.825001 115.825001)
+    (area 79.924999 79.924999 120.075001 120.075001)
     (thickness 1.6)
     (drawings 4)
-    (tracks 174)
+    (tracks 176)
     (zones 0)
     (modules 21)
@@
   )
   (setup
-    (last_trace_width 0.2)
+    (last_trace_width 0.4)
     (user_trace_width 0.15)
     (user_trace_width 0.2)
@@
   )
   (module nRF52:FPC_05P-05mm-RA-SMD_Alt (layer F.Cu)
-    (at 94.2 113.1)
-    (fp_text reference J1 (at 0 1.95) (layer F.SilkS)
+    (at 94.2 117.1)
+    (fp_text reference J1 (at 0 2.25) (layer F.SilkS)
       (effects (font (size 0.5 0.5) (thickness 0.125)))
     )
@@
       (effects (font (size 0.5 0.5) (thickness 0.125)))
     )
-    (fp_line (start -1.25 -1.025) (end 1.25 -1.025) (layer F.SilkS) (width 0.15))
-    (fp_line (start -1.25 1.025) (end 1.25 1.025) (layer F.SilkS) (width 0.15))
-    (fp_line (start -1.25 1.025) (end -1.25 2.45) (layer F.SilkS) (width 0.15))
-    (fp_line (start 1.25 1.025) (end 1.25 2.45) (layer F.SilkS) (width 0.15))
-    (fp_line (start -1.25 2.45) (end -3.8 2.45) (layer F.SilkS) (width 0.15))
-    (fp_line (start 1.25 2.45) (end 3.8 2.45) (layer F.SilkS) (width 0.15))
-    (fp_line (start -3.8 2.45) (end -3.8 0) (layer F.SilkS) (width 0.15))
-    (fp_line (start 3.8 2.45) (end 3.8 0) (layer F.SilkS) (width 0.15))
-    (fp_line (start -3.8 0) (end -1.25 0) (layer F.SilkS) (width 0.15))
-    (fp_line (start 3.8 0) (end 1.25 0) (layer F.SilkS) (width 0.15))
-    (fp_line (start -1.25 0) (end -1.25 -1.025) (layer F.SilkS) (width 0.15))
-    (fp_line (start 1.25 0) (end 1.25 -1.025) (layer F.SilkS) (width 0.15))
+    (fp_line (start -1.55 -1.025) (end 1.55 -1.025) (layer F.SilkS) (width 0.15))
+    (fp_line (start -1.25 1.325) (end 1.25 1.325) (layer F.SilkS) (width 0.15))
+    (fp_line (start -1.25 1.325) (end -1.25 2.75) (layer F.SilkS) (width 0.15))
+    (fp_line (start 1.25 1.325) (end 1.25 2.75) (layer F.SilkS) (width 0.15))
+    (fp_line (start -1.25 2.75) (end -2.55 2.75) (layer F.SilkS) (width 0.15))
+    (fp_line (start 1.25 2.75) (end 2.55 2.75) (layer F.SilkS) (width 0.15))
+    (fp_line (start -2.55 2.75) (end -2.55 0) (layer F.SilkS) (width 0.15))
+    (fp_line (start 2.55 2.75) (end 2.55 0) (layer F.SilkS) (width 0.15))
+    (fp_line (start -2.55 0) (end -1.55 0) (layer F.SilkS) (width 0.15))
+    (fp_line (start 2.55 0) (end 1.55 0) (layer F.SilkS) (width 0.15))
+    (fp_line (start -1.55 0) (end -1.55 -1.025) (layer F.SilkS) (width 0.15))
+    (fp_line (start 1.55 0) (end 1.55 -1.025) (layer F.SilkS) (width 0.15))
     (pad 1 smd rect (at -1 0) (size 0.35 0.8) (layers F.Cu F.Paste F.Mask))
     (pad 2 smd rect (at -0.5 0) (size 0.35 0.8) (layers F.Cu F.Paste F.Mask)
@@
       (net 12 /NFC2))
     (pad 5 smd rect (at 1 0) (size 0.35 0.8) (layers F.Cu F.Paste F.Mask))
-    (pad 0 smd rect (at -2.6 1.3) (size 0.6 2) (layers F.Cu F.Paste F.Mask))
-    (pad 0 smd rect (at 2.6 1.3) (size 0.6 2) (layers F.Cu F.Paste F.Mask))
-  )
-  (gr_line (start 78.75 115.75) (end 78.75 81.75) (angle 90) (layer Edge.Cuts) (width 0.15))
-  (gr_line (start 118.75 115.75) (end 78.75 115.75) (angle 90) (layer Edge.Cuts) (width 0.15))
-  (gr_line (start 118.75 81.75) (end 118.75 115.75) (angle 90) (layer Edge.Cuts) (width 0.15))
-  (gr_line (start 78.75 81.75) (end 118.75 81.75) (angle 90) (layer Edge.Cuts) (width 0.15))
+    (pad 0 smd rect (at -1.9 1.6) (size 0.6 2) (layers F.Cu F.Paste F.Mask))
+    (pad 0 smd rect (at 1.9 1.6) (size 0.6 2) (layers F.Cu F.Paste F.Mask))
+  )
+  (gr_line (start 80 120) (end 80 80) (angle 90) (layer Edge.Cuts) (width 0.15))
+  (gr_line (start 120 120) (end 80 120) (angle 90) (layer Edge.Cuts) (width 0.15))
+  (gr_line (start 120 80) (end 120 120) (angle 90) (layer Edge.Cuts) (width 0.15))
+  (gr_line (start 80 80) (end 120 80) (angle 90) (layer Edge.Cuts) (width 0.15))
+  (segment (start 96.2 104.5) (end 96 104.5) (width 0.4) (layer F.Cu) (net 1))
+  (segment (start 92.55 104.55) (end 92.55 103.7) (width 0.4) (layer F.Cu) (net 1))
+  (segment (start 92.9 104.9) (end 92.55 104.55) (width 0.4) (layer F.Cu) (net 1))
+  (via (at 92.9 104.9) (size 0.41) (drill 0.4) (layers F.Cu B.Cu) (net 1))
+  (segment (start 95.6 104.9) (end 92.9 104.9) (width 0.4) (layer B.Cu) (net 1))
+  (via (at 95.6 104.9) (size 0.41) (drill 0.4) (layers F.Cu B.Cu) (net 1))
+  (segment (start 96 104.5) (end 95.6 104.9) (width 0.4) (layer F.Cu) (net 1))
+  (segment (start 95.75 103.7) (end 95.75 104.15) (width 0.4) (layer F.Cu) (net 1))
+  (segment (start 96.1 104.5) (end 96.2 104.5) (width 0.4) (layer F.Cu) (net 1))
+  (segment (start 96.2 104.5) (end 96.75 104.5) (width 0.4) (layer F.Cu) (net 1))
+  (segment (start 95.75 104.15) (end 96.1 104.5) (width 0.4) (layer F.Cu) (net 1))
   (segment (start 89.65 93.9) (end 89.3 93.9) (width 0.2) (layer F.Cu) (net 1))
   (segment (start 89.1 94.1) (end 89.1 96.5) (width 0.2) (layer F.Cu) (net 1))
   (segment (start 89.3 93.9) (end 89.1 94.1) (width 0.2) (layer F.Cu) (net 1))
   (segment (start 92.55 103.7) (end 90.8 103.7) (width 0.2) (layer F.Cu) (net 1))
+  (segment (start 89.1 102) (end 89.1 96.5) (width 0.2) (layer F.Cu) (net 1))
   (segment (start 90.8 103.7) (end 89.1 102) (width 0.2) (layer F.Cu) (net 1))
-  (segment (start 89.1 102) (end 89.1 96.5) (width 0.2) (layer F.Cu) (net 1))
   (segment (start 89.2 96.4) (end 89.65 96.4) (width 0.2) (layer F.Cu) (net 1))
   (segment (start 89.1 96.5) (end 89.2 96.4) (width 0.2) (layer F.Cu) (net 1))
-  (segment (start 95.75 103.7) (end 95.75 104.65) (width 0.15) (layer F.Cu) (net 1))
-  (segment (start 95.75 104.65) (end 95.8 104.7) (width 0.15) (layer F.Cu) (net 1))
-  (segment (start 92.55 103.7) (end 92.55 104.45) (width 0.15) (layer F.Cu) (net 1))
-  (segment (start 96 104.5) (end 96.75 104.5) (width 0.15) (layer F.Cu) (net 1))
-  (segment (start 95.8 104.7) (end 96 104.5) (width 0.15) (layer F.Cu) (net 1))
-  (via (at 95.8 104.7) (size 0.41) (drill 0.4) (layers F.Cu B.Cu) (net 1))
-  (segment (start 92.8 104.7) (end 95.8 104.7) (width 0.15) (layer B.Cu) (net 1))
-  (via (at 92.8 104.7) (size 0.41) (drill 0.4) (layers F.Cu B.Cu) (net 1))
-  (segment (start 92.55 104.45) (end 92.8 104.7) (width 0.15) (layer F.Cu) (net 1))
   (segment (start 99 97) (end 99 99) (width 0.2) (layer F.Cu) (net 1))
   (segment (start 99 99) (end 100 100) (width 0.2) (layer F.Cu) (net 1))
@@
   (segment (start 104.9 98) (end 104.9 96.9) (width 0.2) (layer F.Cu) (net 10))
   (segment (start 103.9 99) (end 104.9 98) (width 0.2) (layer F.Cu) (net 10))
-  (segment (start 93.7 113.1) (end 93.7 103.75) (width 0.2) (layer F.Cu) (net 11) (status C00000))
-  (segment (start 93.7 103.75) (end 93.65 103.7) (width 0.2) (layer F.Cu) (net 11) (status C00000))
+  (segment (start 93.7 117.1) (end 93.7 103.75) (width 0.2) (layer F.Cu) (net 11) (status 10))
+  (segment (start 93.7 103.75) (end 93.65 103.7) (width 0.2) (layer F.Cu) (net 11))
   (segment (start 93.7 103.75) (end 93.65 103.7) (width 0.2) (layer F.Cu) (net 11))
   (segment (start 97 101.8) (end 95 101.8) (width 0.2) (layer F.Cu) (net 11))
   (segment (start 93.65 103.15) (end 93.65 103.7) (width 0.2) (layer F.Cu) (net 11))
   (segment (start 95 101.8) (end 93.65 103.15) (width 0.2) (layer F.Cu) (net 11))
-  (segment (start 94.7 113.1) (end 94.7 103.75) (width 0.2) (layer F.Cu) (net 12) (status C00000))
-  (segment (start 94.7 103.75) (end 94.65 103.7) (width 0.2) (layer F.Cu) (net 12) (status C00000))
+  (segment (start 94.7 117.1) (end 94.7 103.75) (width 0.2) (layer F.Cu) (net 12) (status 10))
+  (segment (start 94.7 103.75) (end 94.65 103.7) (width 0.2) (layer F.Cu) (net 12))
   (segment (start 94.7 103.75) (end 94.65 103.7) (width 0.2) (layer F.Cu) (net 12))
   (segment (start 97 102.2) (end 95.6 102.2) (width 0.2) (layer F.Cu) (net 12))
