File: nRF52840_reference/kicad/nRF52840_qfaa/nRF52840_qfaa.kicad_pcb (KiCad board)
At the start: 2 copper layers, 38 x 42 mm, 30 parts, among them J1 CONN_COAXIAL, U1 nRF52840, X1 XTAL_32MHZ, X2 XTAL_32KHZ

Commit message: Update KiCAD Project nRF52840_qfaa
Parts:
- removed L2: 10uH, Nordic_misc:L_0603
- removed L3: 15nH, Nordic_misc:L_0402
Connections:
- net Net-(C15-Pad1) renamed /DEC4
- U1 pad B3: Net-(L2-Pad2) -> (no net)
Routing:
- net Net-(L2-Pad2): track 3.54 -> 0.00 mm
- net /DEC4: track 5.99 -> 2.70 mm
- net Net-(L2-Pad1): track 1.36 -> 0.00 mm
