File: nRF52840_reference/kicad/nRF52840_qfaa/nRF52840_qfaa.sch (KiCad schematic (older format))
At the start: 30 parts, among them J1 CONN_COAXIAL, U1 nRF52840, X1 XTAL_32MHZ, X2 XTAL_32KHZ

Commit message: Update KiCAD Project nRF52840_qfaa
Parts:
- removed L2: 10uH, Nordic_misc:L_0603, symbol L
- removed L3: 15nH, Nordic_misc:L_0402, symbol L
Connections:
- net DEC4: now reaches C15.1, U1.B5 (DEC4)
Changed lines of the file:
@@
-$EndComp
-$Comp
-L L L3
-U 1 1 5983C1A6
-P 3600 1250
-F 0 "L3" H 3500 1350 50  0000 C CNN
-F 1 "15nH" H 3500 1250 50  0000 C CNN
-F 2 "Nordic_misc:L_0402" H 3600 1250 50  0001 C CNN
-F 3 "" H 3600 1250 50  0001 C CNN
-	1    3600 1250
-	1    0    0    -1
-$EndComp
-$Comp
-L L L2
-U 1 1 5983C1F7
-P 3600 1700
-F 0 "L2" H 3500 1800 50  0000 C CNN
-F 1 "10uH" H 3500 1700 50  0000 C CNN
-F 2 "Nordic_misc:L_0603" H 3600 1700 50  0001 C CNN
-F 3 "" H 3600 1700 50  0001 C CNN
-	1    3600 1700
-	1    0    0    -1
 $EndComp
 $Comp
@@
 Connection ~ 3200 2000
 Wire Wire Line
-	3600 1400 3600 1550
-Wire Wire Line
-	3700 1850 3700 2550
-Wire Wire Line
 	4100 1600 4100 1750
-Wire Wire Line
-	3600 1100 3600 950
 Wire Wire Line
 	3600 950  4100 950
@@
 	3900 1650 4100 1650
 Connection ~ 4100 1650
-Wire Wire Line
-	3600 1850 3700 1850
 Wire Wire Line
 	5200 1700 5200 1550
@@
 	3500 2450 3200 2450
 Connection ~ 3200 2450
+Text Label 3600 950  2    60   ~ 0
+DEC4
 $EndSCHEMATC
