File: nRF52840_MCU_Board/kicad/PowerSupply.sch (KiCad schematic (older format))
At the start: 9 parts, among them J2 MICROUSB, U2 TLV1117

Commit message: Update KiCAD Project nRF52840_MCU_Board
Parts:
- BATT1: footprint Nordic_misc:keystone_3003 -> Nordic_misc:keystone_3002
Changed lines of the file:
@@
 F 0 "BATT1" H 2650 2950 39  0000 C CNN
 F 1 "CR2032" H 2700 2650 39  0000 C CNN
-F 2 "Nordic_misc:keystone_3003" H 2580 2900 20  0001 C CNN
+F 2 "Nordic_misc:keystone_3002" H 2580 2900 20  0001 C CNN
 F 3 "" H 2550 2750 60  0001 C CNN
 	1    2550 2750
