File: nRF52840_MCU_Board/kicad/nRF52840.sch (KiCad schematic (older format))
At the start: 34 parts, among them J1 CONN_COAXIAL, M1 FPC_05P-RA-SMD, M2 DEBUG_CONNECTOR, U1 nRF52840, X1 XTAL_32KHZ, X2 XTAL_32MHZ

Commit message: Update KiCAD Project nRF52840_MCU_Board
Parts:
- M2: footprint Nordic_misc:Pin_Header_Straight_2x05_Pitch1.27mm_SMD -> Nordic_misc:ftsh-105-01-l-dv
Changed lines of the file:
@@
 F 0 "M2" H 8000 6700 39  0000 C CNN
 F 1 "DEBUG_CONNECTOR" H 8000 6000 39  0000 C CNN
-F 2 "Nordic_misc:Pin_Header_Straight_2x05_Pitch1.27mm_SMD" H 7830 6200 20  0001 C CNN
+F 2 "Nordic_misc:ftsh-105-01-l-dv" H 7830 6200 20  0001 C CNN
 F 3 "" H 7800 6050 60  0001 C CNN
 	1    7800 6050
