File: nRF52840_MCU_Board/kicad/nRF52840_MCU_Board.kicad_pcb (KiCad board)
At the start: 2 copper layers, 45 x 45 mm, 33 parts, among them J1 CONN_COAXIAL, U1 nRF52840, X1 XTAL_32MHZ, X2 XTAL_32KHZ

Commit message: Update KiCAD Project nRF52840_MCU_Board
Parts:
- removed NFC1: NFC_ANTENNA, Nordic_misc:Nordic_misc-NFC_ANT
- added BATT1: CR2032, Nordic_misc:keystone_3003, B.Cu at (39.4, 91.2)
- added C22: 100nF, Capacitors_SMD:C_0402, B.Cu at (54.2, 85.2)
- added C23: 10uF, Capacitors_SMD:C_0603, B.Cu at (55.3, 81.0)
- added C24: 10uF, Capacitors_SMD:C_0603, B.Cu at (60.9, 81.0)
- added C25: 100uF, Capacitors_SMD:C_0805, B.Cu at (53.8, 97.7)
- added J2: MICROUSB, Nordic_misc:conn_usb_B_micro_smd, F.Cu at (96.4, 128.7)
- added J3: Power, Pin_Headers:Pin_Header_Straight_1x08_Pitch2.54mm, F.Cu at (42.8, 128.6)
- added J4: Analog, Pin_Headers:Pin_Header_Straight_1x08_Pitch2.54mm, F.Cu at (65.9, 128.8)
- added J5: Digital3, Pin_Headers:Pin_Header_Straight_2x09_Pitch2.54mm, F.Cu at (109.5, 66.3)
- added J6: Digital0, Pin_Headers:Pin_Header_Straight_1x10_Pitch2.54mm, F.Cu at (44.0, 62.9)
- added J7: Digital1, Pin_Headers:Pin_Header_Straight_1x08_Pitch2.54mm, F.Cu at (71.8, 62.8)
- added J8: Digital2, Pin_Headers:Pin_Header_Straight_1x08_Pitch2.54mm, F.Cu at (93.7, 62.5)
- added M1: FPC_05P-RA-SMD, Nordic_misc:Nordic_misc-FPC_05P-RA-SMD, F.Cu at (108.6, 127.6)
- added M2: DEBUG_CONNECTOR, Nordic_misc:Pin_Header_Straight_2x05_Pitch1.27mm_SMD, F.Cu at (103.6, 110.3)
- added MK1: Mounting_Hole, Nordic_misc:MountingHole_3mm, F.Cu at (34.4, 64.1)
- added MK2: Mounting_Hole, Nordic_misc:MountingHole_3mm, F.Cu at (121.4, 63.5)
- added MK3: Mounting_Hole, Nordic_misc:MountingHole_3mm, F.Cu at (121.6, 128.5)
- added MK4: Mounting_Hole, Nordic_misc:MountingHole_3mm, F.Cu at (33.4, 128.7)
- added R1: 0, Resistors_SMD:R_0402, B.Cu at (59.2, 85.0)
- added R2: 0, Resistors_SMD:R_0402, B.Cu at (60.9, 97.9)
- added U2: TLV1117, TO_SOT_Packages_SMD:SOT-223-3Lead_TabPin2, B.Cu at (59.5, 90.7)
- AE1: footprint Nordic_misc:Nordic_misc-QWMP_BEND_LEFT_+0 -> Nordic_misc:Nordic_misc-QWMP_BEND_RIGHT_+0
- X1: value XTAL_32MHZ -> XTAL_32KHZ; footprint Nordic_nRF:Crystal_SMD_2016-4pin_2.0x1.6mm -> Nordic_nRF:Crystal_SMD_3215-2pin_3.2x1.5mm
- X2: value XTAL_32KHZ -> XTAL_32MHZ; footprint Nordic_nRF:Crystal_SMD_3215-2pin_3.2x1.5mm -> Nordic_nRF:Crystal_SMD_2016-4pin_2.0x1.6mm
- moved C46 13.0 mm to (110.2, 118.4), turned to 0 degrees
- moved C47 13.0 mm to (106.7, 118.2), turned to 0 degrees
Connections:
- C46 pad 1: GND -> /nRF52840/NFC2
- C46 pad 2: /NFC2 -> GND
- C47 pad 1: /NFC1 -> GND
- C47 pad 2: GND -> /nRF52840/NFC1
- U1 pad AA24: (no net) -> Net-(M2-Pad4)
- U1 pad AC13: (no net) -> /nRF52840/P0.18/RESET
- U1 pad AC24: (no net) -> Net-(M2-Pad2)
- U1 pad AD22: (no net) -> /nRF52840/P1.00
- U1 pad AD4: (no net) -> /D-
- U1 pad AD6: (no net) -> /D+
- U1 pad J24: /NFC2 -> /nRF52840/NFC2
- U1 pad L24: /NFC1 -> /nRF52840/NFC1
- X1 pad 1: Net-(C2-Pad2) -> Net-(C16-Pad2)
- X1 pad 2: GND -> Net-(C17-Pad2)
- X2 pad 1: Net-(C16-Pad2) -> Net-(C2-Pad2)
- X2 pad 2: Net-(C17-Pad2) -> GND
Routing:
- net /NFC2: track 14.9 -> 0.00 mm
- net /NFC1: track 12.4 -> 0.00 mm
- net +3V3: track 18.6 -> 15.7 mm
- net GND: track 37.5 -> 39.1 mm
Other:
- board size 45 x 45 mm -> 95 x 72 mm

Commit message: Update KiCAD Project nRF52840_MCU_Board
Parts:
- BATT1: footprint Nordic_misc:keystone_3003 -> Nordic_misc:keystone_3002
- J3, J4, J7, J8: footprint Pin_Headers:Pin_Header_Straight_1x08_Pitch2.54mm -> Nordic_misc:Pin_Header_Straight_1x08_Pitch2.54mm
- J5: footprint Pin_Headers:Pin_Header_Straight_2x09_Pitch2.54mm -> Nordic_misc:Pin_Header_Straight_2x09_Pitch2.54mm
- J6: footprint Pin_Headers:Pin_Header_Straight_1x10_Pitch2.54mm -> Nordic_misc:Pin_Header_Straight_1x10_Pitch2.54mm
- M2: footprint Nordic_misc:Pin_Header_Straight_2x05_Pitch1.27mm_SMD -> Nordic_misc:ftsh-105-01-l-dv
- moved X1 14.2 mm to (92.8, 97.8), turned to 180 degrees
- moved X2 14.0 mm to (105.2, 91.0), turned to 0 degrees
- moved MK3 3.14 mm to (118.5, 128.5)
- moved MK2 2.96 mm to (118.5, 63.5)
- moved M1 0.99 mm to (108.5, 128.6)
- moved C16 0.85 mm to (90.1, 98.0)
- moved C17 0.69 mm to (92.7, 99.6)
- moved C6 0.34 mm to (91.7, 102.4)
- moved C18 0.34 mm to (93.1, 102.4)
- moved L4 0.34 mm to (94.7, 102.3)
- moved BATT1 0.33 mm to (39.7, 91.2)
- moved C1 0.12 mm to (107.2, 91.1)
Connections:
- J2 pad 4: (no net) -> Net-(J2-Pad4)
- J3 pad 1: (no net) -> Net-(J3-Pad1)
- J3 pad 2: (no net) -> Net-(J3-Pad2)
- J3 pad 3: (no net) -> Net-(J3-Pad3)
- J3 pad 4: (no net) -> Net-(J3-Pad4)
- J3 pad 5: (no net) -> Net-(J3-Pad5)
- J3 pad 6: (no net) -> Net-(J3-Pad6)
- J3 pad 7: (no net) -> Net-(J3-Pad7)
- J3 pad 8: (no net) -> Net-(J3-Pad8)
- J4 pad 1: (no net) -> Net-(J4-Pad1)
- J4 pad 2: (no net) -> Net-(J4-Pad2)
- J4 pad 3: (no net) -> Net-(J4-Pad3)
- J4 pad 4: (no net) -> Net-(J4-Pad4)
- J4 pad 5: (no net) -> Net-(J4-Pad5)
- J4 pad 6: (no net) -> Net-(J4-Pad6)
- J4 pad 7: (no net) -> Net-(J4-Pad7)
- J4 pad 8: (no net) -> Net-(J4-Pad8)
- J5 pad 1: (no net) -> Net-(J5-Pad1)
- J5 pad 10: (no net) -> Net-(J5-Pad10)
- J5 pad 11: (no net) -> Net-(J5-Pad11)
- J5 pad 12: (no net) -> Net-(J5-Pad12)
- J5 pad 13: (no net) -> Net-(J5-Pad13)
- J5 pad 14: (no net) -> Net-(J5-Pad14)
- J5 pad 15: (no net) -> Net-(J5-Pad15)
- J5 pad 16: (no net) -> Net-(J5-Pad16)
- J5 pad 17: (no net) -> Net-(J5-Pad17)
- J5 pad 18: (no net) -> Net-(J5-Pad18)
- J5 pad 2: (no net) -> Net-(J5-Pad2)
- J5 pad 3: (no net) -> Net-(J5-Pad3)
- J5 pad 4: (no net) -> Net-(J5-Pad4)
- J5 pad 5: (no net) -> Net-(J5-Pad5)
- J5 pad 6: (no net) -> Net-(J5-Pad6)
- J5 pad 7: (no net) -> Net-(J5-Pad7)
- J5 pad 8: (no net) -> Net-(J5-Pad8)
- J5 pad 9: (no net) -> Net-(J5-Pad9)
- J6 pad 1: (no net) -> Net-(J6-Pad1)
- J6 pad 10: (no net) -> Net-(J6-Pad10)
- J6 pad 2: (no net) -> Net-(J6-Pad2)
- J6 pad 3: (no net) -> Net-(J6-Pad3)
- J6 pad 4: (no net) -> Net-(J6-Pad4)
- J6 pad 5: (no net) -> Net-(J6-Pad5)
- J6 pad 6: (no net) -> Net-(J6-Pad6)
- J6 pad 7: (no net) -> Net-(J6-Pad7)
- J6 pad 8: (no net) -> Net-(J6-Pad8)
- J6 pad 9: (no net) -> Net-(J6-Pad9)
- J7 pad 1: (no net) -> Net-(J7-Pad1)
- J7 pad 2: (no net) -> Net-(J7-Pad2)
- J7 pad 3: (no net) -> Net-(J7-Pad3)
- J7 pad 4: (no net) -> Net-(J7-Pad4)
- J7 pad 5: (no net) -> Net-(J7-Pad5)
- J7 pad 6: (no net) -> Net-(J7-Pad6)
- J7 pad 7: (no net) -> Net-(J7-Pad7)
- J7 pad 8: (no net) -> Net-(J7-Pad8)
- J8 pad 1: (no net) -> Net-(J8-Pad1)
- J8 pad 2: (no net) -> Net-(J8-Pad2)
- J8 pad 3: (no net) -> Net-(J8-Pad3)
- J8 pad 4: (no net) -> Net-(J8-Pad4)
- J8 pad 5: (no net) -> Net-(J8-Pad5)
- J8 pad 6: (no net) -> Net-(J8-Pad6)
- J8 pad 7: (no net) -> Net-(J8-Pad7)
- J8 pad 8: (no net) -> Net-(J8-Pad8)
- M1 pad 1: (no net) -> Net-(M1-Pad1)
- M1 pad 3: (no net) -> Net-(M1-Pad3)
- M1 pad 5: (no net) -> Net-(M1-Pad5)
- M2 pad 7: (no net) -> Net-(M2-Pad7)
- M2 pad 8: (no net) -> Net-(M2-Pad8)
- U1 pad A10: (no net) -> /nRF52840/P0.29
- U1 pad A12: (no net) -> /nRF52840/P0.02
- U1 pad A14: (no net) -> /nRF52840/P1.15
- U1 pad A16: (no net) -> /nRF52840/P1.13
- U1 pad A20: (no net) -> /nRF52840/P1.10
- U1 pad A8: (no net) -> /nRF52840/P0.31
- U1 pad AC11: (no net) -> /nRF52840/P0.16
- U1 pad AC15: (no net) -> /nRF52840/P0.19
- U1 pad AC17: (no net) -> /nRF52840/P0.21
- U1 pad AC19: (no net) -> /nRF52840/P0.23
- U1 pad AC21: (no net) -> /nRF52840/P0.25
- U1 pad AC9: (no net) -> /nRF52840/P0.14
- U1 pad AD10: (no net) -> /nRF52840/P0.15
- U1 pad AD12: (no net) -> /nRF52840/P0.17
- U1 pad AD16: (no net) -> /nRF52840/P0.20
- U1 pad AD18: (no net) -> /nRF52840/P0.22
- U1 pad AD20: (no net) -> /nRF52840/P0.24
- U1 pad AD8: (no net) -> /nRF52840/P0.13
- U1 pad B11: (no net) -> /nRF52840/P0.28
- U1 pad B13: (no net) -> /nRF52840/P0.03
- U1 pad B15: (no net) -> /nRF52840/P1.14
- U1 pad B17: (no net) -> /nRF52840/P1.12
- U1 pad B19: (no net) -> /nRF52840/P1.11
- U1 pad B9: (no net) -> /nRF52840/P0.30
- U1 pad G1: (no net) -> /nRF52840/P0.26
- U1 pad H2: (no net) -> /nRF52840/P0.27
- U1 pad J1: (no net) -> /nRF52840/P0.04/AIN2
- U1 pad K2: (no net) -> /nRF52840/P0.05/AIN3
- U1 pad L1: (no net) -> /nRF52840/P0.06
- U1 pad M2: (no net) -> /nRF52840/P0.07
- U1 pad N1: (no net) -> /nRF52840/P0.08
- U1 pad P2: (no net) -> /nRF52840/P1.08
- U1 pad P23: (no net) -> /nRF52840/P1.07
- U1 pad R1: (no net) -> /nRF52840/P1.09
- U1 pad R24: (no net) -> /nRF52840/P1.06
- U1 pad T2: (no net) -> /nRF52840/P0.11
- U1 pad T23: (no net) -> /nRF52840/P1.05
- U1 pad U1: (no net) -> /nRF52840/P0.12
- U1 pad U24: (no net) -> /nRF52840/P1.04
- U1 pad V23: (no net) -> /nRF52840/P1.03
- U1 pad W24: (no net) -> /nRF52840/P1.02
- U1 pad Y23: (no net) -> /nRF52840/P1.01
Routing:
- net Net-(C16-Pad1): track 8.53 -> 0.02 mm
- net Net-(C17-Pad1): track 7.09 -> 0.05 mm
- net +3V3: track 15.7 -> 8.89 mm
- net Net-(C1-Pad2): track 6.24 -> 0.00 mm
- net VDD: track 6.18 -> 0.00 mm
- net GND: track 39.1 -> 33.1 mm
- net Net-(C2-Pad2): track 4.61 -> 0.00 mm
- net Net-(L4-Pad2): track 3.78 -> 0.00 mm
- net Net-(C17-Pad2): track 2.77 -> 0.00 mm
- net Net-(C16-Pad2): track 1.53 -> 0.00 mm
Other:
- board size 95 x 72 mm -> 92 x 72 mm
