File: nRF52840_MCU_Board/kicad/nRF52840_MCU_Board.sch (KiCad schematic (older format))
At the start: 33 parts, among them J1 CONN_COAXIAL, U1 nRF52840, X1 XTAL_32MHZ, X2 XTAL_32KHZ

Commit message: Update KiCAD Project nRF52840_MCU_Board
Parts:
- removed AE1: Antenna, Nordic_misc:Nordic_misc-QWMP_BEND_LEFT_+0, symbol Antenna
- removed C1, C16, C17, C2: 12pF, Nordic_misc:C_0402, symbol C
- removed C10, C13, C9: N.C, Nordic_misc:C_0402, symbol C
- removed C11: 100pF, Nordic_misc:C_0402, symbol C
- removed C12, C5, C7, C8: 100nF, Nordic_misc:C_0402, symbol C
- removed C14, C15: 1.0uF, Nordic_misc:C_0603, symbol C
- removed C18, C19, C20, C6: 4.7uF, Nordic_misc:C_0603, symbol C
- removed C21: 1.2pF, Nordic_misc:C_0402, symbol C
- removed C3: 0.8pF, Nordic_misc:C_0402, symbol C
- removed C4: 0.5pF, Nordic_misc:C_0402, symbol C
- removed C46, C47: 300pF, Nordic_misc:C_0402, symbol C
- removed J1: CONN_COAXIAL, Nordic_misc:Nordic_misc-MM8130-2600, symbol CONN_COAXIAL
- removed L1: 3.3nH, Nordic_misc:L_0603, symbol L
- removed L2, L4: 10uH, Nordic_misc:L_0603, symbol L
- removed L3: 15nH, Nordic_misc:L_0402, symbol L
- removed NFC1: NFC_ANTENNA, Nordic_misc:Nordic_misc-NFC_ANT, symbol NFC_ANTENNA
- removed U1: nRF52840, Nordic_nRF:AQFN73_7x7mm, symbol nRF52840
- removed X1: XTAL_32MHZ, Nordic_nRF:Crystal_SMD_2016-4pin_2.0x1.6mm, symbol XTAL_32MHZ
- removed X2: XTAL_32KHZ, Nordic_nRF:Crystal_SMD_3215-2pin_3.2x1.5mm, symbol XTAL_32KHZ
- added MK1, MK2, MK3, MK4: Mounting_Hole, Nordic_misc:MountingHole_3mm, symbol Mounting_Hole
