File: nRF52832_reference/kicad/nRF52832_qfaa/nRF52832_qfaa.sch (KiCad schematic (older format))
At the start: 22 parts, among them X1 32MHz, X2 32.768kHz

Commit message: Reference Project nRF52832_qfaa ready
Parts:
- removed L2: 10uH, Inductors_SMD:L_0603, symbol L
- removed L3: 15nH, Inductors_SMD:L_0402, symbol L
Changed lines of the file:
@@
-$EndComp
-$Comp
-L L L2
-U 1 1 59739E09
-P 4750 1450
-F 0 "L2" H 4850 1550 50  0000 C CNN
-F 1 "10uH" H 4900 1400 50  0000 C CNN
-F 2 "Inductors_SMD:L_0603" H 4750 1450 50  0001 C CNN
-F 3 "" H 4750 1450 50  0001 C CNN
-	1    4750 1450
-	1    0    0    -1
-$EndComp
-$Comp
-L L L3
-U 1 1 59739E0A
-P 4750 1050
-F 0 "L3" H 4850 1150 50  0000 C CNN
-F 1 "15nH" H 4900 1000 50  0000 C CNN
-F 2 "Inductors_SMD:L_0402" H 4750 1050 50  0001 C CNN
-F 3 "" H 4750 1050 50  0001 C CNN
-	1    4750 1050
-	1    0    0    -1
 $EndComp
 $Comp
@@
 Connection ~ 7500 3450
 Wire Wire Line
-	4750 1200 4750 1300
-Wire Wire Line
-	4750 1600 4750 1700
-Wire Wire Line
-	4750 1700 4950 1700
-Wire Wire Line
-	4950 1700 4950 2150
-Wire Wire Line
 	4750 750  5350 750
-Wire Wire Line
-	4750 750  4750 900
 Wire Wire Line
 	5350 1050 5350 1150
@@
 Text Label 7450 1500 0    60   ~ 0
 DEC2
-Text Label 5050 750  0    60   ~ 0
+Text Label 4750 750  0    60   ~ 0
 DEC4
 Wire Wire Line

Commit message: Update nRF52832_reference
Parts:
- X1: footprint Crystals:Crystal_SMD_2016-4pin_2.0x1.6mm -> Nordic_nRF:Crystal_SMD_2016-4pin_2.0x1.6mm
- X2: footprint Crystals:Crystal_SMD_3215-2pin_3.2x1.5mm -> Nordic_nRF:Crystal_SMD_3215-2pin_3.2x1.5mm
- nRF1: footprint nRF52:UQFN-48-1EP_6x6mm_Pitch0.4mm -> Nordic_nRF:Nordic_nRF-QFN40P600X600X90-48_N
Changed lines of the file:
@@
 LIBS:Nordic_nRF
 LIBS:nRF52832_qfaa-cache
-EELAYER 25 0
+EELAYER 26 0
 EELAYER END
 $Descr USLetter 11000 8500
@@
 F 0 "X2" V 2500 2950 50  0000 C CNN
 F 1 "32.768kHz" V 2650 3050 50  0000 C CNN
-F 2 "Crystals:Crystal_SMD_3215-2pin_3.2x1.5mm" H 2550 2800 50  0001 C CNN
+F 2 "Nordic_nRF:Crystal_SMD_3215-2pin_3.2x1.5mm" H 2550 2800 50  0001 C CNN
 F 3 "" H 2550 2800 50  0001 C CNN
 	1    2550 2800
@@
 F 0 "X1" V 8450 2500 50  0000 L CNN
 F 1 "32MHz" V 8550 2300 50  0000 L CNN
-F 2 "Crystals:Crystal_SMD_2016-4pin_2.0x1.6mm" H 8650 2700 50  0001 C CNN
+F 2 "Nordic_nRF:Crystal_SMD_2016-4pin_2.0x1.6mm" H 8650 2700 50  0001 C CNN
 F 3 "" H 8650 2700 50  0001 C CNN
 	1    8650 2700
@@
 F 0 "nRF1" H 5400 3600 60  0000 C CNN
 F 1 "nRF52832" H 5400 3400 60  0000 C CNN
-F 2 "nRF52:UQFN-48-1EP_6x6mm_Pitch0.4mm" H 5400 3400 60  0001 C CNN
+F 2 "Nordic_nRF:Nordic_nRF-QFN40P600X600X90-48_N" H 5400 3400 60  0001 C CNN
 F 3 "" H 5400 3400 60  0001 C CNN
 	1    5400 3400
