File: nRF52832_reference/kicad/nRF52832_qfaa_dcdc/nRF52832_qfaa_dcdc.kicad_pcb (KiCad board)
At the start: 2 copper layers, 45 x 85 mm, 25 parts, among them X1 32MHz, X2 32.768kHz

Commit message: Reference Project nRF52832_qfaa_dcdc ready
Parts:
- removed C13, C14: TBD, Capacitors_SMD:C_0402
- removed NFC1: NFC_ANTENNA, Nordic_misc:Nordic_misc-NFC_ANT
- moved MK2 45.0 mm to (116.7, 116.6)
- moved MK1 44.8 mm to (78.3, 116.7)
Connections:
- nRF1 pad 11: /NFC1 -> /P0.09
- nRF1 pad 12: /NFC2 -> /P0.10
Routing:
- net /NFC1: track 7.67 -> 0.00 mm
- net /NFC2: track 6.63 -> 0.00 mm
- net GND: track 100.9 -> 100.3 mm, vias 2 -> 0
Other:
- board size 45 x 85 mm -> 45 x 40 mm

Commit message: Update nRF52832_reference
Parts:
- X1: footprint Crystals:Crystal_SMD_2016-4pin_2.0x1.6mm -> Nordic_nRF:Crystal_SMD_2016-4pin_2.0x1.6mm
- X2: footprint Crystals:Crystal_SMD_3215-2pin_3.2x1.5mm -> Nordic_nRF:Crystal_SMD_3215-2pin_3.2x1.5mm
- nRF1: footprint nRF52:UQFN-48-1EP_6x6mm_Pitch0.4mm -> Nordic_nRF:Nordic_nRF-QFN40P600X600X90-48_N
Connections:
- L1 pad 2: /RF -> (no net)
