File: nRF52832_reference/kicad/nRF52832_qfaa_dcdc/nRF52832_qfaa_dcdc.sch (KiCad schematic (older format))
At the start: 25 parts, among them X1 32MHz, X2 32.768kHz

Commit message: Reference Project nRF52832_qfaa_dcdc ready
Parts:
- removed C13, C14: TBD, Capacitors_SMD:C_0402, symbol C
- removed NFC1: NFC_ANTENNA, Nordic_misc:Nordic_misc-NFC_ANT, symbol NFC_ANTENNA
Connections:
- net NFC1 renamed P0.09
- net NFC2 renamed P0.10
- no-connect marks 1 -> 0
Changed lines of the file:
@@
 	3800 3150 4150 3150
-Wire Wire Line
-	2550 3950 4150 3950
-Wire Wire Line
-	2550 3850 4150 3850
 Wire Wire Line
 	3800 3750 4150 3750
@@
 Wire Wire Line
 	8450 2700 8400 2700
-$Comp
-L C C13
-U 1 1 59739E12
-P 2900 3600
-F 0 "C13" H 2700 3700 50  0000 L CNN
-F 1 "TBD" H 2700 3500 50  0000 L CNN
-F 2 "Capacitors_SMD:C_0402" H 2938 3450 50  0001 C CNN
-F 3 "" H 2900 3600 50  0001 C CNN
-	1    2900 3600
-	-1   0    0    -1
-$EndComp
-Wire Wire Line
-	2900 3750 2900 3850
-$Comp
-L C C14
-U 1 1 59739E13
-P 2900 4200
-F 0 "C14" H 2700 4300 50  0000 L CNN
-F 1 "TBD" H 2700 4100 50  0000 L CNN
-F 2 "Capacitors_SMD:C_0402" H 2938 4050 50  0001 C CNN
-F 3 "" H 2900 4200 50  0001 C CNN
-	1    2900 4200
-	-1   0    0    -1
-$EndComp
-Wire Wire Line
-	2900 4050 2900 3950
-Connection ~ 2900 3850
-Connection ~ 2900 3950
-Text Label 3200 3950 2    60   ~ 0
-NFC2
-Text Label 3200 3850 2    60   ~ 0
-NFC1
-$Comp
-L GND-RESCUE-nRF52832_qfaa_dcdc #PWR013
-U 1 1 59739E14
-P 2900 4450
-F 0 "#PWR013" H 2900 4200 50  0001 C CNN
-F 1 "GND" H 2900 4300 50  0000 C CNN
-F 2 "" H 2900 4450 50  0001 C CNN
-F 3 "" H 2900 4450 50  0001 C CNN
-	1    2900 4450
-	-1   0    0    -1
-$EndComp
-Wire Wire Line
-	2900 4450 2900 4350
-$Comp
-L GND-RESCUE-nRF52832_qfaa_dcdc #PWR014
-U 1 1 59739E15
-P 2900 3350
-F 0 "#PWR014" H 2900 3100 50  0001 C CNN
-F 1 "GND" H 2900 3200 50  0000 C CNN
-F 2 "" H 2900 3350 50  0001 C CNN
-F 3 "" H 2900 3350 50  0001 C CNN
-	1    2900 3350
-	1    0    0    1
-$EndComp
-Wire Wire Line
-	2900 3350 2900 3450
 Text HLabel 8200 3450 2    60   BiDi ~ 0
 RF
@@
 	7250 3150 6650 3150
 $Comp
-L GND-RESCUE-nRF52832_qfaa_dcdc #PWR015
+L GND-RESCUE-nRF52832_qfaa_dcdc #PWR013
 U 1 1 5973CAAA
 P 7450 2000
-F 0 "#PWR015" H 7450 1750 50  0001 C CNN
+F 0 "#PWR013" H 7450 1750 50  0001 C CNN
 F 1 "GND" H 7450 1850 50  0000 C CNN
 F 2 "" H 7450 2000 50  0001 C CNN
@@
 DEC1
 $Comp
-L +3.3V-RESCUE-nRF52832_qfaa_dcdc #PWR016
+L +3.3V-RESCUE-nRF52832_qfaa_dcdc #PWR014
 U 1 1 5973FB66
 P 4200 1450
-F 0 "#PWR016" H 4200 1300 50  0001 C CNN
+F 0 "#PWR014" H 4200 1300 50  0001 C CNN
 F 1 "+3.3V" H 4200 1590 50  0000 C CNN
 F 2 "" H 4200 1450 50  0001 C CNN
@@
 $EndComp
 $Comp
-L +3.3V-RESCUE-nRF52832_qfaa_dcdc #PWR017
+L +3.3V-RESCUE-nRF52832_qfaa_dcdc #PWR015
 U 1 1 5973FC37
 P 1800 1700
-F 0 "#PWR017" H 1800 1550 50  0001 C CNN
+F 0 "#PWR015" H 1800 1550 50  0001 C CNN
 F 1 "+3.3V" H 1800 1840 50  0000 C CNN
 F 2 "" H 1800 1700 50  0001 C CNN
@@
 $EndComp
 $Comp
-L +3.3V-RESCUE-nRF52832_qfaa_dcdc #PWR018
+L +3.3V-RESCUE-nRF52832_qfaa_dcdc #PWR016
 U 1 1 5973FE1C
 P 4150 4750
-F 0 "#PWR018" H 4150 4600 50  0001 C CNN
+F 0 "#PWR016" H 4150 4600 50  0001 C CNN
 F 1 "+3.3V" H 4150 4890 50  0000 C CNN
 F 2 "" H 4150 4750 50  0001 C CNN
@@
 $EndComp
 $Comp
-L +3.3V-RESCUE-nRF52832_qfaa_dcdc #PWR019
+L +3.3V-RESCUE-nRF52832_qfaa_dcdc #PWR017
 U 1 1 5973FF85
 P 6200 1400
-F 0 "#PWR019" H 6200 1250 50  0001 C CNN
+F 0 "#PWR017" H 6200 1250 50  0001 C CNN
 F 1 "+3.3V" H 6200 1540 50  0000 C CNN
 F 2 "" H 6200 1400 50  0001 C CNN
@@
 	4750 2050 4200 2050
 Connection ~ 4200 2050
-NoConn ~ 2550 3700
 $Comp
 L Mounting_Hole MK1
@@
 	1    0    0    -1
 $EndComp
-$Comp
-L NFC_ANTENNA NFC1
-U 1 1 597D020B
-P 2050 3750
-F 0 "NFC1" H 2050 3700 39  0000 C CNN
-F 1 "NFC_ANTENNA" H 2150 4120 45  0000 R TNN
-F 2 "Nordic_misc:Nordic_misc-NFC_ANT" H 2080 3900 20  0001 C CNN
-F 3 "" H 2050 3750 60  0001 C CNN
-	1    2050 3750
-	-1   0    0    1
-$EndComp
+Text HLabel 3800 3950 0    60   BiDi ~ 0
+P0.10
+Text HLabel 3800 3850 0    60   BiDi ~ 0
+P0.09
+Wire Wire Line
+	3800 3850 4150 3850
+Wire Wire Line
+	4150 3950 3800 3950
 $EndSCHEMATC

Commit message: Update nRF52832_reference
Parts:
- X1: footprint Crystals:Crystal_SMD_2016-4pin_2.0x1.6mm -> Nordic_nRF:Crystal_SMD_2016-4pin_2.0x1.6mm
- X2: footprint Crystals:Crystal_SMD_3215-2pin_3.2x1.5mm -> Nordic_nRF:Crystal_SMD_3215-2pin_3.2x1.5mm
- nRF1: footprint nRF52:UQFN-48-1EP_6x6mm_Pitch0.4mm -> Nordic_nRF:Nordic_nRF-QFN40P600X600X90-48_N
Changed lines of the file:
@@
 LIBS:Nordic_nRF
 LIBS:nRF52832_qfaa_dcdc-cache
-EELAYER 25 0
+EELAYER 26 0
 EELAYER END
 $Descr USLetter 11000 8500
@@
 F 0 "X2" V 2500 2950 50  0000 C CNN
 F 1 "32.768kHz" V 2650 3050 50  0000 C CNN
-F 2 "Crystals:Crystal_SMD_3215-2pin_3.2x1.5mm" H 2550 2800 50  0001 C CNN
+F 2 "Nordic_nRF:Crystal_SMD_3215-2pin_3.2x1.5mm" H 2550 2800 50  0001 C CNN
 F 3 "" H 2550 2800 50  0001 C CNN
 	1    2550 2800
@@
 F 0 "X1" V 8450 2500 50  0000 L CNN
 F 1 "32MHz" V 8550 2300 50  0000 L CNN
-F 2 "Crystals:Crystal_SMD_2016-4pin_2.0x1.6mm" H 8650 2700 50  0001 C CNN
+F 2 "Nordic_nRF:Crystal_SMD_2016-4pin_2.0x1.6mm" H 8650 2700 50  0001 C CNN
 F 3 "" H 8650 2700 50  0001 C CNN
 	1    8650 2700
@@
 F 0 "nRF1" H 5400 3600 60  0000 C CNN
 F 1 "nRF52832" H 5400 3400 60  0000 C CNN
-F 2 "nRF52:UQFN-48-1EP_6x6mm_Pitch0.4mm" H 5400 3400 60  0001 C CNN
+F 2 "Nordic_nRF:Nordic_nRF-QFN40P600X600X90-48_N" H 5400 3400 60  0001 C CNN
 F 3 "" H 5400 3400 60  0001 C CNN
 	1    5400 3400
