File: nRF52832_MCU_Board/kicad/PowerSupply.sch (KiCad schematic (older format))
At the start: 9 parts, among them J5 MICROUSB, U2 TLV1117

Commit message: Update KiCad Projec nRF52832_MCU_Board
Parts:
- J5: footprint w_conn_pc:conn_usb_B_micro_smd -> Nordic_misc:conn_usb_B_micro_smd
Connections:
- net +3V3: no longer BATT1.2 (+), R13.2
- new net +3.3VP: BATT1.2 (+), R13.2
Changed lines of the file:
@@
 $Descr USLetter 11000 8500
 encoding utf-8
-Sheet 3 3
+Sheet 3 4
 Title ""
 Date ""
@@
 $EndComp
 $Comp
-L GND #PWR024
+L GND #PWR01
 U 1 1 597D2A05
 P 3950 2800
-F 0 "#PWR024" H 3950 2550 50  0001 C CNN
+F 0 "#PWR01" H 3950 2550 50  0001 C CNN
 F 1 "GND" H 3950 2650 50  0000 C CNN
 F 2 "" H 3950 2800 50  0001 C CNN
@@
 $EndComp
 $Comp
-L GND #PWR025
+L GND #PWR02
 U 1 1 597D2A3A
 P 4250 2800
-F 0 "#PWR025" H 4250 2550 50  0001 C CNN
+F 0 "#PWR02" H 4250 2550 50  0001 C CNN
 F 1 "GND" H 4250 2650 50  0000 C CNN
 F 2 "" H 4250 2800 50  0001 C CNN
@@
 $EndComp
 $Comp
-L GND #PWR026
+L GND #PWR03
 U 1 1 597D2A54
 P 5750 2800
-F 0 "#PWR026" H 5750 2550 50  0001 C CNN
+F 0 "#PWR03" H 5750 2550 50  0001 C CNN
 F 1 "GND" H 5750 2650 50  0000 C CNN
 F 2 "" H 5750 2800 50  0001 C CNN
@@
 $EndComp
 $Comp
-L GND #PWR027
+L GND #PWR04
 U 1 1 597D2AA5
 P 6050 2800
-F 0 "#PWR027" H 6050 2550 50  0001 C CNN
+F 0 "#PWR04" H 6050 2550 50  0001 C CNN
 F 1 "GND" H 6050 2650 50  0000 C CNN
 F 2 "" H 6050 2800 50  0001 C CNN
@@
 $EndComp
 $Comp
-L GND #PWR028
+L GND #PWR05
 U 1 1 597D2ABF
 P 5000 2800
-F 0 "#PWR028" H 5000 2550 50  0001 C CNN
+F 0 "#PWR05" H 5000 2550 50  0001 C CNN
 F 1 "GND" H 5000 2650 50  0000 C CNN
 F 2 "" H 5000 2800 50  0001 C CNN
@@
 $EndComp
 $Comp
-L +5V #PWR029
+L +5V #PWR06
 U 1 1 597D30A3
 P 3700 2250
-F 0 "#PWR029" H 3700 2100 50  0001 C CNN
+F 0 "#PWR06" H 3700 2100 50  0001 C CNN
 F 1 "+5V" H 3700 2390 50  0000 C CNN
 F 2 "" H 3700 2250 50  0001 C CNN
@@
 Connection ~ 3950 2300
 $Comp
-L +3.3V #PWR030
+L +3.3V #PWR07
 U 1 1 597D30F2
 P 6150 2250
-F 0 "#PWR030" H 6150 2100 50  0001 C CNN
+F 0 "#PWR07" H 6150 2100 50  0001 C CNN
 F 1 "+3.3V" H 6150 2390 50  0000 C CNN
 F 2 "" H 6150 2250 50  0001 C CNN
@@
 Connection ~ 6050 2300
 $Comp
-L PWR_FLAG #FLG031
+L PWR_FLAG #FLG08
 U 1 1 597D3131
 P 6350 2150
-F 0 "#FLG031" H 6350 2225 50  0001 C CNN
+F 0 "#FLG08" H 6350 2225 50  0001 C CNN
 F 1 "PWR_FLAG" H 6350 2300 50  0000 C CNN
 F 2 "" H 6350 2150 50  0001 C CNN
@@
 Connection ~ 6150 2300
 $Comp
-L PWR_FLAG #FLG032
+L PWR_FLAG #FLG09
 U 1 1 597D317F
 P 3500 2200
-F 0 "#FLG032" H 3500 2275 50  0001 C CNN
+F 0 "#FLG09" H 3500 2275 50  0001 C CNN
 F 1 "PWR_FLAG" H 3500 2350 50  0000 C CNN
 F 2 "" H 3500 2200 50  0001 C CNN
@@
 F 0 "J5" H 1650 3550 39  0000 C CNN
 F 1 "MICROUSB" H 1400 2830 39  0000 C CNN
-F 2 "w_conn_pc:conn_usb_B_micro_smd" H 1430 3050 20  0001 C CNN
+F 2 "Nordic_misc:conn_usb_B_micro_smd" H 1430 3050 20  0001 C CNN
 F 3 "" H 1400 2900 60  0001 C CNN
 	1    1400 2900
@@
 NoConn ~ 1600 2700
 $Comp
-L GND #PWR033
+L GND #PWR010
 U 1 1 597D3BFA
 P 1650 2950
-F 0 "#PWR033" H 1650 2700 50  0001 C CNN
+F 0 "#PWR010" H 1650 2700 50  0001 C CNN
 F 1 "GND" H 1650 2800 50  0000 C CNN
 F 2 "" H 1650 2950 50  0001 C CNN
@@
 $EndComp
 $Comp
-L +5VD #PWR034
+L +5VD #PWR011
 U 1 1 597D3C2A
 P 1700 2250
-F 0 "#PWR034" H 1700 2100 50  0001 C CNN
+F 0 "#PWR011" H 1700 2100 50  0001 C CNN
 F 1 "+5VD" H 1700 2390 50  0000 C CNN
 F 2 "" H 1700 2250 50  0001 C CNN
@@
 	1700 2400 1700 2250
 $Comp
-L +5V #PWR035
+L +5V #PWR012
 U 1 1 597D3C8A
 P 2150 2250
-F 0 "#PWR035" H 2150 2100 50  0001 C CNN
+F 0 "#PWR012" H 2150 2100 50  0001 C CNN
 F 1 "+5V" H 2150 2390 50  0000 C CNN
 F 2 "" H 2150 2250 50  0001 C CNN
@@
 	2150 2400 2150 2250
 $Comp
-L PWR_FLAG #FLG036
+L PWR_FLAG #FLG013
 U 1 1 597D3DA0
 P 1550 2150
-F 0 "#FLG036" H 1550 2225 50  0001 C CNN
+F 0 "#FLG013" H 1550 2225 50  0001 C CNN
 F 1 "PWR_FLAG" H 1550 2300 50  0000 C CNN
 F 2 "" H 1550 2150 50  0001 C CNN
@@
 	2400 2400 2800 2400
 $Comp
-L GND #PWR037
+L GND #PWR014
 U 1 1 597D3F23
 P 2550 3150
-F 0 "#PWR037" H 2550 2900 50  0001 C CNN
+F 0 "#PWR014" H 2550 2900 50  0001 C CNN
 F 1 "GND" H 2550 3000 50  0000 C CNN
 F 2 "" H 2550 3150 50  0001 C CNN
@@
 	2550 3150 2550 3050
 $Comp
-L +3V3 #PWR038
-U 1 1 597D40BA
-P 2550 2250
-F 0 "#PWR038" H 2550 2100 50  0001 C CNN
-F 1 "+3V3" H 2550 2390 50  0000 C CNN
-F 2 "" H 2550 2250 50  0001 C CNN
-F 3 "" H 2550 2250 50  0001 C CNN
-	1    2550 2250
-	1    0    0    -1
-$EndComp
-$Comp
-L PWR_FLAG #FLG039
+L PWR_FLAG #FLG015
 U 1 1 597D4126
 P 2400 2150
-F 0 "#FLG039" H 2400 2225 50  0001 C CNN
+F 0 "#FLG015" H 2400 2225 50  0001 C CNN
 F 1 "PWR_FLAG" H 2400 2300 50  0000 C CNN
 F 2 "" H 2400 2150 50  0001 C CNN
@@
 Connection ~ 2550 2400
 $Comp
-L +3.3V #PWR040
+L +3.3V #PWR016
 U 1 1 597D423B
 P 3200 2250
-F 0 "#PWR040" H 3200 2100 50  0001 C CNN
+F 0 "#PWR016" H 3200 2100 50  0001 C CNN
 F 1 "+3.3V" H 3200 2390 50  0000 C CNN
 F 2 "" H 3200 2250 50  0001 C CNN
@@
 Wire Wire Line
 	3200 2400 3100 2400
+$Comp
+L +3.3VP #PWR017
+U 1 1 597D52F4
+P 2550 2250
+F 0 "#PWR017" H 2700 2200 50  0001 C CNN
+F 1 "+3.3VP" H 2550 2350 50  0000 C CNN
+F 2 "" H 2550 2250 50  0001 C CNN
+F 3 "" H 2550 2250 50  0001 C CNN
+	1    2550 2250
+	1    0    0    -1
+$EndComp
+Text HLabel 7400 1550 2    60   Output ~ 0
+VDD
+Text HLabel 7400 1850 2    60   Output ~ 0
+5V
+$Comp
+L +3.3V #PWR018
+U 1 1 597E4BDB
+P 7300 1450
+F 0 "#PWR018" H 7300 1300 50  0001 C CNN
+F 1 "+3.3V" H 7300 1590 50  0000 C CNN
+F 2 "" H 7300 1450 50  0001 C CNN
+F 3 "" H 7300 1450 50  0001 C CNN
+	1    7300 1450
+	1    0    0    -1
+$EndComp
+Wire Wire Line
+	7300 1450 7300 1550
+Wire Wire Line
+	7300 1550 7400 1550
+$Comp
+L +5V #PWR019
+U 1 1 597E4CB2
+P 7300 1750
+F 0 "#PWR019" H 7300 1600 50  0001 C CNN
+F 1 "+5V" H 7300 1890 50  0000 C CNN
+F 2 "" H 7300 1750 50  0001 C CNN
+F 3 "" H 7300 1750 50  0001 C CNN
+	1    7300 1750
+	1    0    0    -1
+$EndComp
+Wire Wire Line
+	7400 1850 7300 1850
+Wire Wire Line
+	7300 1850 7300 1750
 $EndSCHEMATC

Commit message: Update KiCAD Project nRF52832_MCU_Board
Parts:
- BATT1: footprint Nordic_misc:keystone_3000 -> Nordic_misc:Keystone_1058_1x2032-CoinCell
Changed lines of the file:
@@
 F 0 "BATT1" H 2650 2950 39  0000 C CNN
 F 1 "CR1632" H 2700 2650 39  0000 C CNN
-F 2 "Nordic_misc:keystone_3000" H 2580 2900 20  0001 C CNN
+F 2 "Nordic_misc:Keystone_1058_1x2032-CoinCell" H 2580 2900 20  0001 C CNN
 F 3 "" H 2550 2750 60  0001 C CNN
 	1    2550 2750

Commit message: Update  KiCAD Project nRF52832_MCU_Board
Parts:
- BATT1: footprint Nordic_misc:Keystone_1058_1x2032-CoinCell -> w_battery_holders:keystone_3000
- U2: footprint TO_SOT_Packages_SMD:TO-263-3Lead -> TO_SOT_Packages_SMD:SOT-223-3Lead_TabPin2
Changed lines of the file:
@@
 $Descr USLetter 11000 8500
 encoding utf-8
-Sheet 3 4
+Sheet 2 4
 Title ""
 Date ""
@@
 F 0 "U2" H 5100 2430 39  0000 C CNN
 F 1 "TLV1117" H 4600 2920 45  0000 L BNN
-F 2 "TO_SOT_Packages_SMD:TO-263-3Lead" H 4630 2650 20  0001 C CNN
+F 2 "TO_SOT_Packages_SMD:SOT-223-3Lead_TabPin2" H 4630 2650 20  0001 C CNN
 F 3 "" H 4600 2500 60  0001 C CNN
 	1    4600 2500
@@
 F 0 "BATT1" H 2650 2950 39  0000 C CNN
 F 1 "CR1632" H 2700 2650 39  0000 C CNN
-F 2 "Nordic_misc:Keystone_1058_1x2032-CoinCell" H 2580 2900 20  0001 C CNN
+F 2 "w_battery_holders:keystone_3000" H 2580 2900 20  0001 C CNN
 F 3 "" H 2550 2750 60  0001 C CNN
 	1    2550 2750

Commit message: Update KiCAD Project nRF52832_MCU_Board
Parts:
- BATT1: value CR1632 -> CR2032; footprint w_battery_holders:keystone_3000 -> Nordic_misc:keystone_3003
Changed lines of the file:
@@
 EESchema Schematic File Version 2
-LIBS:nRF52832_MCU_Board-rescue
 LIBS:Nordic_misc
 LIBS:Nordic_nRF
@@
 P 2550 2750
 F 0 "BATT1" H 2650 2950 39  0000 C CNN
-F 1 "CR1632" H 2700 2650 39  0000 C CNN
-F 2 "w_battery_holders:keystone_3000" H 2580 2900 20  0001 C CNN
+F 1 "CR2032" H 2700 2650 39  0000 C CNN
+F 2 "Nordic_misc:keystone_3003" H 2580 2900 20  0001 C CNN
 F 3 "" H 2550 2750 60  0001 C CNN
 	1    2550 2750
