File: nRF52832_MCU_Board/kicad/nRF528323_MCU.sch (KiCad schematic (older format))
At the start: 30 parts, among them J6 DEBUG_CONNECTOR, J7 CONN_01X05, X1 32MHz, X2 32.768kHz

Commit message: Update WIP
Parts:
- added ANT1: Antenna, Nordic_misc:Nordic_misc-QWMP_MEANDERED_LEFT_+6, symbol Antenna
- added C13: N.C, Capacitors_SMD:C_0402, symbol C
- added C20: TBD, Capacitors_SMD:C_0402, symbol C
- added J8: MM8130-2600, Connectors:SMA_SMD_Jack_Straight, symbol CONN_COAXIAL
- J6: footprint (none) -> Pin_Headers:Pin_Header_Straight_2x05_Pitch2.54mm_SMD
- J7: footprint (none) -> Nordic_misc:Nordic_misc-FPC_05P-RA-SMD
- R1, R2, R3, R4: footprint (none) -> Resistors_SMD:R_0402
- gave numbers to parts that had none: 5
Connections:
- net GND: now also C13.1, C20.1
- net RF: no longer names the net of L1.2
- net RF: now also C13.2
- new net: ANT1.1 (A), C20.2, J8.2 (Ext)
Other:
- moved on the sheet: C3, L1

Commit message: Update KiCad Projec nRF52832_MCU_Board
Parts:
- J6: footprint Pin_Headers:Pin_Header_Straight_2x05_Pitch2.54mm_SMD -> Nordic_misc:Pin_Header_Straight_2x05_Pitch1.27mm_SMD
- J8: footprint Connectors:SMA_SMD_Jack_Straight -> Nordic_misc:Nordic_misc-MM8130-2600
Changed lines of the file:
@@
 $Descr USLetter 11000 8500
 encoding utf-8
-Sheet 2 2
+Sheet 2 4
 Title ""
 Date "2017-07-22"
@@
 VDD_nRF
 $Comp
-L PWR_FLAG #FLG01
+L PWR_FLAG #FLG042
 U 1 1 597D1430
 P 2150 1700
-F 0 "#FLG01" H 2150 1775 50  0001 C CNN
+F 0 "#FLG042" H 2150 1775 50  0001 C CNN
 F 1 "PWR_FLAG" H 2150 1850 50  0000 C CNN
 F 2 "" H 2150 1700 50  0001 C CNN
@@
 $EndComp
 $Comp
-L GND-RESCUE-nRF52832_qfaa_nfc #PWR02
+L GND-RESCUE-nRF52832_qfaa_nfc #PWR043
 U 1 1 597D1432
 P 4200 2100
-F 0 "#PWR02" H 4200 1850 50  0001 C CNN
+F 0 "#PWR043" H 4200 1850 50  0001 C CNN
 F 1 "GND" H 4200 1950 50  0000 C CNN
 F 2 "" H 4200 2100 50  0001 C CNN
@@
 $EndComp
 $Comp
-L GND-RESCUE-nRF52832_qfaa_nfc #PWR03
+L GND-RESCUE-nRF52832_qfaa_nfc #PWR044
 U 1 1 597D1434
 P 3650 2100
-F 0 "#PWR03" H 3650 1850 50  0001 C CNN
+F 0 "#PWR044" H 3650 1850 50  0001 C CNN
 F 1 "GND" H 3650 1950 50  0000 C CNN
 F 2 "" H 3650 2100 50  0001 C CNN
@@
 $EndComp
 $Comp
-L GND-RESCUE-nRF52832_qfaa_nfc #PWR04
+L GND-RESCUE-nRF52832_qfaa_nfc #PWR045
 U 1 1 597D1436
 P 4150 5350
-F 0 "#PWR04" H 4150 5100 50  0001 C CNN
+F 0 "#PWR045" H 4150 5100 50  0001 C CNN
 F 1 "GND" H 4150 5200 50  0000 C CNN
 F 2 "" H 4150 5350 50  0001 C CNN
@@
 $EndComp
 $Comp
-L GND-RESCUE-nRF52832_qfaa_nfc #PWR05
+L GND-RESCUE-nRF52832_qfaa_nfc #PWR046
 U 1 1 597D1438
 P 6200 2000
-F 0 "#PWR05" H 6200 1750 50  0001 C CNN
+F 0 "#PWR046" H 6200 1750 50  0001 C CNN
 F 1 "GND" H 6200 1850 50  0000 C CNN
 F 2 "" H 6200 2000 50  0001 C CNN
@@
 $EndComp
 $Comp
-L GND-RESCUE-nRF52832_qfaa_nfc #PWR06
+L GND-RESCUE-nRF52832_qfaa_nfc #PWR047
 U 1 1 597D143C
 P 1350 3150
-F 0 "#PWR06" H 1350 2900 50  0001 C CNN
+F 0 "#PWR047" H 1350 2900 50  0001 C CNN
 F 1 "GND" H 1350 3000 50  0000 C CNN
 F 2 "" H 1350 3150 50  0001 C CNN
@@
 $EndComp
 $Comp
-L GND-RESCUE-nRF52832_qfaa_nfc #PWR07
+L GND-RESCUE-nRF52832_qfaa_nfc #PWR048
 U 1 1 597D143F
 P 9450 3150
-F 0 "#PWR07" H 9450 2900 50  0001 C CNN
+F 0 "#PWR048" H 9450 2900 50  0001 C CNN
 F 1 "GND" H 9450 3000 50  0000 C CNN
 F 2 "" H 9450 3150 50  0001 C CNN
@@
 $EndComp
 $Comp
-L GND-RESCUE-nRF52832_qfaa_nfc #PWR08
+L GND-RESCUE-nRF52832_qfaa_nfc #PWR049
 U 1 1 597D1442
 P 6950 2000
-F 0 "#PWR08" H 6950 1750 50  0001 C CNN
+F 0 "#PWR049" H 6950 1750 50  0001 C CNN
 F 1 "GND" H 6950 1850 50  0000 C CNN
 F 2 "" H 6950 2000 50  0001 C CNN
@@
 $EndComp
 $Comp
-L GND-RESCUE-nRF52832_qfaa_nfc #PWR09
+L GND-RESCUE-nRF52832_qfaa_nfc #PWR050
 U 1 1 597D1444
 P 8250 3950
-F 0 "#PWR09" H 8250 3700 50  0001 C CNN
+F 0 "#PWR050" H 8250 3700 50  0001 C CNN
 F 1 "GND" H 8250 3800 50  0000 C CNN
 F 2 "" H 8250 3950 50  0001 C CNN
@@
 $EndComp
 $Comp
-L GND-RESCUE-nRF52832_qfaa_nfc #PWR010
+L GND-RESCUE-nRF52832_qfaa_nfc #PWR051
 U 1 1 597D1449
 P 5350 1150
-F 0 "#PWR010" H 5350 900 50  0001 C CNN
+F 0 "#PWR051" H 5350 900 50  0001 C CNN
 F 1 "GND" H 5350 1000 50  0000 C CNN
 F 2 "" H 5350 1150 50  0001 C CNN
@@
 $EndComp
 $Comp
-L GND-RESCUE-nRF52832_qfaa_nfc #PWR011
+L GND-RESCUE-nRF52832_qfaa_nfc #PWR052
 U 1 1 597D144B
 P 8900 2700
-F 0 "#PWR011" H 8900 2450 50  0001 C CNN
+F 0 "#PWR052" H 8900 2450 50  0001 C CNN
 F 1 "GND" H 8900 2550 50  0000 C CNN
 F 2 "" H 8900 2700 50  0001 C CNN
@@
 	8900 2700 8850 2700
 $Comp
-L GND-RESCUE-nRF52832_qfaa_nfc #PWR012
+L GND-RESCUE-nRF52832_qfaa_nfc #PWR053
 U 1 1 597D144C
 P 8400 2700
-F 0 "#PWR012" H 8400 2450 50  0001 C CNN
+F 0 "#PWR053" H 8400 2450 50  0001 C CNN
 F 1 "GND" H 8400 2550 50  0000 C CNN
 F 2 "" H 8400 2700 50  0001 C CNN
@@
 NFC1
 $Comp
-L GND-RESCUE-nRF52832_qfaa_nfc #PWR013
+L GND-RESCUE-nRF52832_qfaa_nfc #PWR054
 U 1 1 597D144F
 P 1900 5050
-F 0 "#PWR013" H 1900 4800 50  0001 C CNN
+F 0 "#PWR054" H 1900 4800 50  0001 C CNN
 F 1 "GND" H 1900 4900 50  0000 C CNN
 F 2 "" H 1900 5050 50  0001 C CNN
@@
 	1900 5050 1900 5000
 $Comp
-L GND-RESCUE-nRF52832_qfaa_nfc #PWR014
+L GND-RESCUE-nRF52832_qfaa_nfc #PWR055
 U 1 1 597D1450
 P 1900 3700
-F 0 "#PWR014" H 1900 3450 50  0001 C CNN
+F 0 "#PWR055" H 1900 3450 50  0001 C CNN
 F 1 "GND" H 1900 3550 50  0000 C CNN
 F 2 "" H 1900 3700 50  0001 C CNN
@@
 	7250 3150 6650 3150
 $Comp
-L GND-RESCUE-nRF52832_qfaa_nfc #PWR015
+L GND-RESCUE-nRF52832_qfaa_nfc #PWR056
 U 1 1 597D1452
 P 7450 2000
-F 0 "#PWR015" H 7450 1750 50  0001 C CNN
+F 0 "#PWR056" H 7450 1750 50  0001 C CNN
 F 1 "GND" H 7450 1850 50  0000 C CNN
 F 2 "" H 7450 2000 50  0001 C CNN
@@
 DEC1
 $Comp
-L +3.3V-RESCUE-nRF52832_qfaa_nfc #PWR016
+L +3.3V-RESCUE-nRF52832_qfaa_nfc #PWR057
 U 1 1 597D1453
 P 4200 1450
-F 0 "#PWR016" H 4200 1300 50  0001 C CNN
+F 0 "#PWR057" H 4200 1300 50  0001 C CNN
 F 1 "+3.3V" H 4200 1590 50  0000 C CNN
 F 2 "" H 4200 1450 50  0001 C CNN
@@
 $EndComp
 $Comp
-L +3.3V-RESCUE-nRF52832_qfaa_nfc #PWR017
+L +3.3V-RESCUE-nRF52832_qfaa_nfc #PWR058
 U 1 1 597D1454
 P 1800 1700
-F 0 "#PWR017" H 1800 1550 50  0001 C CNN
+F 0 "#PWR058" H 1800 1550 50  0001 C CNN
 F 1 "+3.3V" H 1800 1840 50  0000 C CNN
 F 2 "" H 1800 1700 50  0001 C CNN
@@
 $EndComp
 $Comp
-L +3.3V-RESCUE-nRF52832_qfaa_nfc #PWR018
+L +3.3V-RESCUE-nRF52832_qfaa_nfc #PWR059
 U 1 1 597D1455
 P 4150 4750
-F 0 "#PWR018" H 4150 4600 50  0001 C CNN
+F 0 "#PWR059" H 4150 4600 50  0001 C CNN
 F 1 "+3.3V" H 4150 4890 50  0000 C CNN
 F 2 "" H 4150 4750 50  0001 C CNN
@@
 $EndComp
 $Comp
-L +3.3V-RESCUE-nRF52832_qfaa_nfc #PWR019
+L +3.3V-RESCUE-nRF52832_qfaa_nfc #PWR060
 U 1 1 597D1456
 P 6200 1400
-F 0 "#PWR019" H 6200 1250 50  0001 C CNN
+F 0 "#PWR060" H 6200 1250 50  0001 C CNN
 F 1 "+3.3V" H 6200 1540 50  0000 C CNN
 F 2 "" H 6200 1400 50  0001 C CNN
@@
 F 0 "J6" H 7500 5200 50  0000 C CNN
 F 1 "DEBUG_CONNECTOR" H 7500 4600 50  0000 C CNN
-F 2 "Pin_Headers:Pin_Header_Straight_2x05_Pitch2.54mm_SMD" H 7500 3700 50  0001 C CNN
+F 2 "Nordic_misc:Pin_Header_Straight_2x05_Pitch1.27mm_SMD" H 7500 3700 50  0001 C CNN
 F 3 "" H 7500 3700 50  0001 C CNN
 	1    7500 4900
@@
 P0.21/RESET
 $Comp
-L GND #PWR020
+L GND #PWR061
 U 1 1 597D6B06
 P 7900 5500
-F 0 "#PWR020" H 7900 5250 50  0001 C CNN
+F 0 "#PWR061" H 7900 5250 50  0001 C CNN
 F 1 "GND" H 7900 5350 50  0000 C CNN
 F 2 "" H 7900 5500 50  0001 C CNN
@@
 Connection ~ 7900 5100
 $Comp
-L +3.3V-RESCUE-nRF52832_qfaa_nfc #PWR021
+L +3.3V-RESCUE-nRF52832_qfaa_nfc #PWR062
 U 1 1 597D6E8B
 P 7900 4600
-F 0 "#PWR021" H 7900 4450 50  0001 C CNN
+F 0 "#PWR062" H 7900 4450 50  0001 C CNN
 F 1 "+3.3V" H 7900 4740 50  0000 C CNN
 F 2 "" H 7900 4600 50  0001 C CNN
@@
 F 0 "J8" H 9160 3570 50  0000 C CNN
 F 1 "MM8130-2600" H 9500 3450 50  0000 C CNN
-F 2 "Connectors:SMA_SMD_Jack_Straight" H 9150 3450 50  0001 C CNN
+F 2 "Nordic_misc:Nordic_misc-MM8130-2600" H 9150 3450 50  0001 C CNN
 F 3 "" H 9150 3450 50  0001 C CNN
 	1    9150 3450
@@
 $EndComp
 $Comp
-L GND #PWR022
+L GND #PWR063
 U 1 1 597D3163
 P 9150 4200
-F 0 "#PWR022" H 9150 3950 50  0001 C CNN
+F 0 "#PWR063" H 9150 3950 50  0001 C CNN
 F 1 "GND" H 9150 4050 50  0000 C CNN
 F 2 "" H 9150 4200 50  0001 C CNN
@@
 	9150 3800 9150 3650
 $Comp
-L GND #PWR023
+L GND #PWR064
 U 1 1 597D337A
 P 8850 3950
-F 0 "#PWR023" H 8850 3700 50  0001 C CNN
+F 0 "#PWR064" H 8850 3700 50  0001 C CNN
 F 1 "GND" H 8850 3800 50  0000 C CNN
 F 2 "" H 8850 3950 50  0001 C CNN

Commit message: Update KiCad Project nRF52832_MCU_Board
Parts:
- J6: footprint Nordic_misc:Pin_Header_Straight_2x05_Pitch1.27mm_SMD -> Nordic_misc:ftsh-105-01-l-dv
Changed lines of the file:
@@
 F 0 "J6" H 7500 5200 50  0000 C CNN
 F 1 "DEBUG_CONNECTOR" H 7500 4600 50  0000 C CNN
-F 2 "Nordic_misc:Pin_Header_Straight_2x05_Pitch1.27mm_SMD" H 7500 3700 50  0001 C CNN
+F 2 "Nordic_misc:ftsh-105-01-l-dv" H 7500 3700 50  0001 C CNN
 F 3 "" H 7500 3700 50  0001 C CNN
 	1    7500 4900

Commit message: Update KiCAD Project nRF52832_MCU_Board
Parts:
- X1: footprint Crystals:Crystal_SMD_2016-4pin_2.0x1.6mm -> Nordic_nRF:Crystal_SMD_2016-4pin_2.0x1.6mm
- X2: footprint Crystals:Crystal_SMD_3215-2pin_3.2x1.5mm -> Nordic_nRF:Crystal_SMD_3215-2pin_3.2x1.5mm
Changed lines of the file:
@@
 $Descr USLetter 11000 8500
 encoding utf-8
-Sheet 2 4
+Sheet 4 4
 Title ""
 Date "2017-07-22"
@@
 F 0 "X2" V 2000 2950 50  0000 C CNN
 F 1 "32.768kHz" V 2150 3050 50  0000 C CNN
-F 2 "Crystals:Crystal_SMD_3215-2pin_3.2x1.5mm" H 2050 2800 50  0001 C CNN
+F 2 "Nordic_nRF:Crystal_SMD_3215-2pin_3.2x1.5mm" H 2050 2800 50  0001 C CNN
 F 3 "" H 2050 2800 50  0001 C CNN
 	1    2050 2800
@@
 F 0 "X1" V 8450 2500 50  0000 L CNN
 F 1 "32MHz" V 8550 2300 50  0000 L CNN
-F 2 "Crystals:Crystal_SMD_2016-4pin_2.0x1.6mm" H 8650 2700 50  0001 C CNN
+F 2 "Nordic_nRF:Crystal_SMD_2016-4pin_2.0x1.6mm" H 8650 2700 50  0001 C CNN
 F 3 "" H 8650 2700 50  0001 C CNN
 	1    8650 2700

Commit message: Update KiCAD Project nRF52832_MCU_Board
Parts:
- J6: value DEBUG_CONNECTOR -> CONN_02X05
- nRF1: footprint nRF52:UQFN-48-1EP_6x6mm_Pitch0.4mm -> Nordic_nRF:Nordic_nRF-QFN40P600X600X90-48_N
Connections:
- net +3V3: now also J6.2 (P2); no longer J6.1 (P1)
- net GND: now also J6.10 (P10), J6.6 (P6); no longer J6.5 (P5), J6.9 (P9)
- net P0.18/SWO/2.2B: now also J6.5 (P5); no longer J6.6 (P6)
- net P0.21/RESET/2.2B: now also J6.9 (P9); no longer J6.10 (P10)
- net SWCLK: now also J6.3 (P3); no longer J6.4 (P4)
- net SWDIO: now also J6.1 (P1); no longer J6.2 (P2)
- no-connect marks 3 -> 6
Changed lines of the file:
@@
 EESchema Schematic File Version 2
-LIBS:power
-LIBS:device
-LIBS:transistors
-LIBS:conn
-LIBS:linear
-LIBS:regul
+LIBS:nRF52832_MCU_Board-rescue
+LIBS:Nordic_misc
+LIBS:Nordic_nRF
+LIBS:74xgxx
 LIBS:74xx
-LIBS:cmos4000
-LIBS:adc-dac
-LIBS:memory
-LIBS:xilinx
-LIBS:microcontrollers
-LIBS:dsp
-LIBS:microchip
-LIBS:analog_switches
-LIBS:motorola
-LIBS:texas
-LIBS:intel
-LIBS:audio
-LIBS:interface
-LIBS:digital-audio
-LIBS:philips
-LIBS:display
-LIBS:cypress
-LIBS:siliconi
-LIBS:opto
-LIBS:atmel
-LIBS:contrib
-LIBS:valves
-LIBS:74xgxx
 LIBS:ac-dc
 LIBS:actel
+LIBS:adc-dac
 LIBS:allegro
 LIBS:Altera
 LIBS:analog_devices
+LIBS:analog_switches
+LIBS:atmel
+LIBS:audio
 LIBS:battery_management
 LIBS:bbd
@@
 LIBS:brooktre
 LIBS:cmos_ieee
+LIBS:cmos4000
+LIBS:conn
+LIBS:contrib
+LIBS:cypress
 LIBS:dc-dc
+LIBS:device
+LIBS:digital-audio
 LIBS:diode
+LIBS:display
+LIBS:dsp
 LIBS:elec-unifil
 LIBS:ESD_Protection
@@
 LIBS:graphic
 LIBS:hc11
+LIBS:intel
+LIBS:interface
 LIBS:ir
 LIBS:Lattice
 LIBS:leds
+LIBS:linear
 LIBS:logo
 LIBS:maxim
 LIBS:mechanical
+LIBS:memory
+LIBS:microchip
 LIBS:microchip_dspic33dsc
 LIBS:microchip_pic10mcu
@@
 LIBS:microchip_pic24mcu
 LIBS:microchip_pic32mcu
+LIBS:microcontrollers
 LIBS:modules
 LIBS:motor_drivers
+LIBS:motorola
 LIBS:motors
 LIBS:msp430
@@
 LIBS:nxp_armmcu
 LIBS:onsemi
-LIBS:OPA4134
+LIBS:opto
 LIBS:Oscillators
-LIBS:PCM3168A
+LIBS:philips
+LIBS:power
+LIBS:Power_Management
 LIBS:powerint
-LIBS:Power_Management
 LIBS:pspice
 LIBS:references
+LIBS:regul
 LIBS:relays
 LIBS:rfcom
 LIBS:sensors
 LIBS:silabs
+LIBS:siliconi
 LIBS:stm8
 LIBS:stm32
 LIBS:supertex
 LIBS:switches
-LIBS:TMS320VC5502
+LIBS:texas
 LIBS:transf
+LIBS:transistors
 LIBS:triac_thyristor
-LIBS:TS3A27518E
 LIBS:ttl_ieee
+LIBS:valves
 LIBS:video
 LIBS:w_analog
-LIBS:w_connectors
 LIBS:w_device
-LIBS:wiznet
 LIBS:w_logic
 LIBS:w_memory
 LIBS:w_microcontrollers
 LIBS:w_opto
-LIBS:Worldsemi
 LIBS:w_relay
 LIBS:w_rtx
 LIBS:w_transistor
 LIBS:w_vacuum
+LIBS:wiznet
+LIBS:Worldsemi
 LIBS:Xicor
+LIBS:xilinx
 LIBS:zetex
 LIBS:Zilog
-LIBS:Nordic_misc
-LIBS:Nordic_nRF
 LIBS:nRF52832_MCU_Board-cache
 EELAYER 25 0
@@
 F 0 "nRF1" H 5400 3600 60  0000 C CNN
 F 1 "nRF52832" H 5400 3400 60  0000 C CNN
-F 2 "nRF52:UQFN-48-1EP_6x6mm_Pitch0.4mm" H 5400 3400 60  0001 C CNN
+F 2 "Nordic_nRF:Nordic_nRF-QFN40P600X600X90-48_N" H 5400 3400 60  0001 C CNN
 F 3 "" H 5400 3400 60  0001 C CNN
 	1    5400 3400
@@
 Wire Wire Line
 	6900 3850 6900 4700
-$Comp
-L CONN_02X05 J6
-U 1 1 597D61D5
-P 7500 4900
-F 0 "J6" H 7500 5200 50  0000 C CNN
-F 1 "DEBUG_CONNECTOR" H 7500 4600 50  0000 C CNN
-F 2 "Nordic_misc:ftsh-105-01-l-dv" H 7500 3700 50  0001 C CNN
-F 3 "" H 7500 3700 50  0001 C CNN
-	1    7500 4900
-	-1   0    0    -1
-$EndComp
 Wire Wire Line
 	6900 4700 7250 4700
@@
 U 1 1 597D20DE
 P 9150 3450
+AR Path="/597D20DE" Ref="J8"  Part="1"
+AR Path="/597D109B/597D20DE" Ref="J8"  Part="1"
 F 0 "J8" H 9160 3570 50  0000 C CNN
 F 1 "MM8130-2600" H 9500 3450 50  0000 C CNN
@@
 	9900 3700 9150 3700
 Connection ~ 9150 3700
+$Comp
+L CONN_02X05 J6
+U 1 1 597F8B91
+P 7500 4900
+F 0 "J6" H 7500 5200 39  0000 C CNN
+F 1 "CONN_02X05" H 7500 4600 39  0000 C CNN
+F 2 "Nordic_misc:ftsh-105-01-l-dv" H 7500 3700 50  0001 C CNN
+F 3 "" H 7500 3700 50  0001 C CNN
+	1    7500 4900
+	1    0    0    -1
+$EndComp
+NoConn ~ 7750 4800
+NoConn ~ 7750 5000
+NoConn ~ 7250 5000
 $EndSCHEMATC

Commit message: Update  KiCAD Project nRF52832_MCU_Board
Connections:
- net at C13.2, L1.2: now also J8.1 (In)
Other:
- moved on the sheet: C20, J8
Changed lines of the file:
@@
 VDD_nRF
 $Comp
-L PWR_FLAG #FLG042
+L PWR_FLAG #FLG040
 U 1 1 597D1430
 P 2150 1700
-F 0 "#FLG042" H 2150 1775 50  0001 C CNN
+F 0 "#FLG040" H 2150 1775 50  0001 C CNN
 F 1 "PWR_FLAG" H 2150 1850 50  0000 C CNN
 F 2 "" H 2150 1700 50  0001 C CNN
@@
 $EndComp
 $Comp
-L GND-RESCUE-nRF52832_qfaa_nfc #PWR043
+L GND-RESCUE-nRF52832_qfaa_nfc #PWR041
 U 1 1 597D1432
 P 4200 2100
-F 0 "#PWR043" H 4200 1850 50  0001 C CNN
+F 0 "#PWR041" H 4200 1850 50  0001 C CNN
 F 1 "GND" H 4200 1950 50  0000 C CNN
 F 2 "" H 4200 2100 50  0001 C CNN
@@
 $EndComp
 $Comp
-L GND-RESCUE-nRF52832_qfaa_nfc #PWR044
+L GND-RESCUE-nRF52832_qfaa_nfc #PWR042
 U 1 1 597D1434
 P 3650 2100
-F 0 "#PWR044" H 3650 1850 50  0001 C CNN
+F 0 "#PWR042" H 3650 1850 50  0001 C CNN
 F 1 "GND" H 3650 1950 50  0000 C CNN
 F 2 "" H 3650 2100 50  0001 C CNN
@@
 $EndComp
 $Comp
-L GND-RESCUE-nRF52832_qfaa_nfc #PWR045
+L GND-RESCUE-nRF52832_qfaa_nfc #PWR043
 U 1 1 597D1436
 P 4150 5350
-F 0 "#PWR045" H 4150 5100 50  0001 C CNN
+F 0 "#PWR043" H 4150 5100 50  0001 C CNN
 F 1 "GND" H 4150 5200 50  0000 C CNN
 F 2 "" H 4150 5350 50  0001 C CNN
@@
 $EndComp
 $Comp
-L GND-RESCUE-nRF52832_qfaa_nfc #PWR046
+L GND-RESCUE-nRF52832_qfaa_nfc #PWR044
 U 1 1 597D1438
 P 6200 2000
-F 0 "#PWR046" H 6200 1750 50  0001 C CNN
+F 0 "#PWR044" H 6200 1750 50  0001 C CNN
 F 1 "GND" H 6200 1850 50  0000 C CNN
 F 2 "" H 6200 2000 50  0001 C CNN
@@
 $EndComp
 $Comp
-L GND-RESCUE-nRF52832_qfaa_nfc #PWR047
+L GND-RESCUE-nRF52832_qfaa_nfc #PWR045
 U 1 1 597D143C
 P 1350 3150
-F 0 "#PWR047" H 1350 2900 50  0001 C CNN
+F 0 "#PWR045" H 1350 2900 50  0001 C CNN
 F 1 "GND" H 1350 3000 50  0000 C CNN
 F 2 "" H 1350 3150 50  0001 C CNN
@@
 $EndComp
 $Comp
-L GND-RESCUE-nRF52832_qfaa_nfc #PWR048
+L GND-RESCUE-nRF52832_qfaa_nfc #PWR046
 U 1 1 597D143F
 P 9450 3150
-F 0 "#PWR048" H 9450 2900 50  0001 C CNN
+F 0 "#PWR046" H 9450 2900 50  0001 C CNN
 F 1 "GND" H 9450 3000 50  0000 C CNN
 F 2 "" H 9450 3150 50  0001 C CNN
@@
 $EndComp
 $Comp
-L GND-RESCUE-nRF52832_qfaa_nfc #PWR049
+L GND-RESCUE-nRF52832_qfaa_nfc #PWR047
 U 1 1 597D1442
 P 6950 2000
-F 0 "#PWR049" H 6950 1750 50  0001 C CNN
+F 0 "#PWR047" H 6950 1750 50  0001 C CNN
 F 1 "GND" H 6950 1850 50  0000 C CNN
 F 2 "" H 6950 2000 50  0001 C CNN
@@
 $EndComp
 $Comp
-L GND-RESCUE-nRF52832_qfaa_nfc #PWR050
+L GND-RESCUE-nRF52832_qfaa_nfc #PWR048
 U 1 1 597D1444
 P 8250 3950
-F 0 "#PWR050" H 8250 3700 50  0001 C CNN
+F 0 "#PWR048" H 8250 3700 50  0001 C CNN
 F 1 "GND" H 8250 3800 50  0000 C CNN
 F 2 "" H 8250 3950 50  0001 C CNN
@@
 $EndComp
 $Comp
-L GND-RESCUE-nRF52832_qfaa_nfc #PWR051
+L GND-RESCUE-nRF52832_qfaa_nfc #PWR049
 U 1 1 597D1449
 P 5350 1150
-F 0 "#PWR051" H 5350 900 50  0001 C CNN
+F 0 "#PWR049" H 5350 900 50  0001 C CNN
 F 1 "GND" H 5350 1000 50  0000 C CNN
 F 2 "" H 5350 1150 50  0001 C CNN
@@
 $EndComp
 $Comp
-L GND-RESCUE-nRF52832_qfaa_nfc #PWR052
+L GND-RESCUE-nRF52832_qfaa_nfc #PWR050
 U 1 1 597D144B
 P 8900 2700
-F 0 "#PWR052" H 8900 2450 50  0001 C CNN
+F 0 "#PWR050" H 8900 2450 50  0001 C CNN
 F 1 "GND" H 8900 2550 50  0000 C CNN
 F 2 "" H 8900 2700 50  0001 C CNN
@@
 	8900 2700 8850 2700
 $Comp
-L GND-RESCUE-nRF52832_qfaa_nfc #PWR053
+L GND-RESCUE-nRF52832_qfaa_nfc #PWR051
 U 1 1 597D144C
 P 8400 2700
-F 0 "#PWR053" H 8400 2450 50  0001 C CNN
+F 0 "#PWR051" H 8400 2450 50  0001 C CNN
 F 1 "GND" H 8400 2550 50  0000 C CNN
 F 2 "" H 8400 2700 50  0001 C CNN
@@
 NFC1
 $Comp
-L GND-RESCUE-nRF52832_qfaa_nfc #PWR054
+L GND-RESCUE-nRF52832_qfaa_nfc #PWR052
 U 1 1 597D144F
 P 1900 5050
-F 0 "#PWR054" H 1900 4800 50  0001 C CNN
+F 0 "#PWR052" H 1900 4800 50  0001 C CNN
 F 1 "GND" H 1900 4900 50  0000 C CNN
 F 2 "" H 1900 5050 50  0001 C CNN
@@
 	1900 5050 1900 5000
 $Comp
-L GND-RESCUE-nRF52832_qfaa_nfc #PWR055
+L GND-RESCUE-nRF52832_qfaa_nfc #PWR053
 U 1 1 597D1450
 P 1900 3700
-F 0 "#PWR055" H 1900 3450 50  0001 C CNN
+F 0 "#PWR053" H 1900 3450 50  0001 C CNN
 F 1 "GND" H 1900 3550 50  0000 C CNN
 F 2 "" H 1900 3700 50  0001 C CNN
@@
 	7250 3150 6650 3150
 $Comp
-L GND-RESCUE-nRF52832_qfaa_nfc #PWR056
+L GND-RESCUE-nRF52832_qfaa_nfc #PWR054
 U 1 1 597D1452
 P 7450 2000
-F 0 "#PWR056" H 7450 1750 50  0001 C CNN
+F 0 "#PWR054" H 7450 1750 50  0001 C CNN
 F 1 "GND" H 7450 1850 50  0000 C CNN
 F 2 "" H 7450 2000 50  0001 C CNN
@@
 DEC1
 $Comp
-L +3.3V-RESCUE-nRF52832_qfaa_nfc #PWR057
+L +3.3V-RESCUE-nRF52832_qfaa_nfc #PWR055
 U 1 1 597D1453
 P 4200 1450
-F 0 "#PWR057" H 4200 1300 50  0001 C CNN
+F 0 "#PWR055" H 4200 1300 50  0001 C CNN
 F 1 "+3.3V" H 4200 1590 50  0000 C CNN
 F 2 "" H 4200 1450 50  0001 C CNN
@@
 $EndComp
 $Comp
-L +3.3V-RESCUE-nRF52832_qfaa_nfc #PWR058
+L +3.3V-RESCUE-nRF52832_qfaa_nfc #PWR056
 U 1 1 597D1454
 P 1800 1700
-F 0 "#PWR058" H 1800 1550 50  0001 C CNN
+F 0 "#PWR056" H 1800 1550 50  0001 C CNN
 F 1 "+3.3V" H 1800 1840 50  0000 C CNN
 F 2 "" H 1800 1700 50  0001 C CNN
@@
 $EndComp
 $Comp
-L +3.3V-RESCUE-nRF52832_qfaa_nfc #PWR059
+L +3.3V-RESCUE-nRF52832_qfaa_nfc #PWR057
 U 1 1 597D1455
 P 4150 4750
-F 0 "#PWR059" H 4150 4600 50  0001 C CNN
+F 0 "#PWR057" H 4150 4600 50  0001 C CNN
 F 1 "+3.3V" H 4150 4890 50  0000 C CNN
 F 2 "" H 4150 4750 50  0001 C CNN
@@
 $EndComp
 $Comp
-L +3.3V-RESCUE-nRF52832_qfaa_nfc #PWR060
+L +3.3V-RESCUE-nRF52832_qfaa_nfc #PWR058
 U 1 1 597D1456
 P 6200 1400
-F 0 "#PWR060" H 6200 1250 50  0001 C CNN
+F 0 "#PWR058" H 6200 1250 50  0001 C CNN
 F 1 "+3.3V" H 6200 1540 50  0000 C CNN
 F 2 "" H 6200 1400 50  0001 C CNN
@@
 P0.21/RESET
 $Comp
-L GND #PWR061
+L GND #PWR059
 U 1 1 597D6B06
 P 7900 5500
-F 0 "#PWR061" H 7900 5250 50  0001 C CNN
+F 0 "#PWR059" H 7900 5250 50  0001 C CNN
 F 1 "GND" H 7900 5350 50  0000 C CNN
 F 2 "" H 7900 5500 50  0001 C CNN
@@
 Connection ~ 7900 5100
 $Comp
-L +3.3V-RESCUE-nRF52832_qfaa_nfc #PWR062
+L +3.3V-RESCUE-nRF52832_qfaa_nfc #PWR060
 U 1 1 597D6E8B
 P 7900 4600
-F 0 "#PWR062" H 7900 4450 50  0001 C CNN
+F 0 "#PWR060" H 7900 4450 50  0001 C CNN
 F 1 "+3.3V" H 7900 4740 50  0000 C CNN
 F 2 "" H 7900 4600 50  0001 C CNN
@@
 L CONN_COAXIAL J8
 U 1 1 597D20DE
-P 9150 3450
+P 9200 3450
 AR Path="/597D20DE" Ref="J8"  Part="1"
 AR Path="/597D109B/597D20DE" Ref="J8"  Part="1"
-F 0 "J8" H 9160 3570 50  0000 C CNN
-F 1 "MM8130-2600" H 9500 3450 50  0000 C CNN
-F 2 "Nordic_misc:Nordic_misc-MM8130-2600" H 9150 3450 50  0001 C CNN
-F 3 "" H 9150 3450 50  0001 C CNN
-	1    9150 3450
-	1    0    0    -1
-$EndComp
-Wire Wire Line
-	8750 3450 9000 3450
-Wire Wire Line
-	8850 3450 8850 3550
-Connection ~ 8850 3450
+F 0 "J8" H 9210 3570 50  0000 C CNN
+F 1 "MM8130-2600" H 9550 3450 50  0000 C CNN
+F 2 "Nordic_misc:Nordic_misc-MM8130-2600" H 9200 3450 50  0001 C CNN
+F 3 "" H 9200 3450 50  0001 C CNN
+	1    9200 3450
+	1    0    0    -1
+$EndComp
 $Comp
 L C C20
 U 1 1 597D2E58
-P 9150 3950
-F 0 "C20" H 9000 3850 50  0000 L CNN
-F 1 "TBD" H 9000 4050 50  0000 L CNN
-F 2 "Capacitors_SMD:C_0402" H 9188 3800 50  0001 C CNN
-F 3 "" H 9150 3950 50  0001 C CNN
-	1    9150 3950
+P 9200 4050
+F 0 "C20" H 9050 3950 50  0000 L CNN
+F 1 "TBD" H 9050 4150 50  0000 L CNN
+F 2 "Capacitors_SMD:C_0402" H 9238 3900 50  0001 C CNN
+F 3 "" H 9200 4050 50  0001 C CNN
+	1    9200 4050
 	-1   0    0    1
 $EndComp
 $Comp
-L GND #PWR063
+L GND #PWR061
 U 1 1 597D3163
-P 9150 4200
-F 0 "#PWR063" H 9150 3950 50  0001 C CNN
-F 1 "GND" H 9150 4050 50  0000 C CNN
-F 2 "" H 9150 4200 50  0001 C CNN
-F 3 "" H 9150 4200 50  0001 C CNN
-	1    9150 4200
-	1    0    0    -1
-$EndComp
-Wire Wire Line
-	9150 4200 9150 4100
-Wire Wire Line
-	9150 3800 9150 3650
-$Comp
-L GND #PWR064
+P 9200 4300
+F 0 "#PWR061" H 9200 4050 50  0001 C CNN
+F 1 "GND" H 9200 4150 50  0000 C CNN
+F 2 "" H 9200 4300 50  0001 C CNN
+F 3 "" H 9200 4300 50  0001 C CNN
+	1    9200 4300
+	1    0    0    -1
+$EndComp
+Wire Wire Line
+	9200 4300 9200 4200
+Wire Wire Line
+	9200 3700 9200 3900
+$Comp
+L GND #PWR062
 U 1 1 597D337A
 P 8850 3950
-F 0 "#PWR064" H 8850 3700 50  0001 C CNN
+F 0 "#PWR062" H 8850 3700 50  0001 C CNN
 F 1 "GND" H 8850 3800 50  0000 C CNN
 F 2 "" H 8850 3950 50  0001 C CNN
@@
 $EndComp
 Wire Wire Line
-	9900 3550 9900 3700
-Wire Wire Line
-	9900 3700 9150 3700
-Connection ~ 9150 3700
+	9900 3550 9900 3800
+Wire Wire Line
+	9900 3800 9200 3800
+Connection ~ 9200 3800
 $Comp
 L CONN_02X05 J6
@@
 NoConn ~ 7750 5000
 NoConn ~ 7250 5000
+Wire Wire Line
+	8750 3450 9000 3450
+Wire Wire Line
+	8850 3550 8850 3450
+Connection ~ 8850 3450
 $EndSCHEMATC
